Commit message: Add additional mounting points for accessories, fix the position of the existing front_mount

File: dingo_description/urdf/dingo-d.urdf.xacro (robot description, xacro)
@@ -156,9 +156,42 @@
     <child link="imu_link" />
   </joint>
+  <!--
+    Mounting points for accessories in the top channel.
+    These are flush with the top of the robot and all oriented to face forwards
+  -->
   <link name="front_mount"></link>
   <joint name="front_mount_joint" type="fixed">
-    <origin xyz="0.2 0 0.05" rpy="0 0 0" />
+    <origin xyz="0.2 0 0.068" rpy="0 0 0" />
     <parent link="chassis_link"/>
     <child link="front_mount" />
+  </joint>
+  <link name="mid_mount"></link>
+  <joint name="mid_mount_joint" type="fixed">
+    <origin xyz="0 0 0.067" rpy="0 0 0" />
+    <parent link="chassis_link"/>
+    <child link="mid_mount" />
+  </joint>
+  <link name="rear_mount"></link>
+  <joint name="rear_mount_joint" type="fixed">
+    <origin xyz="-0.2 0 0.068" rpy="0 0 0" />
+    <parent link="chassis_link"/>
+    <child link="rear_mount" />
+  </joint>
+  <!--
+    Mounting points for accessories on the front/rear bumpers.
+    Use with caution, but thin sensors (e.g Raspberry Pi NoIR camera) could
+    be mounted here for low-budget, front/rear-facing capabilities
+  -->
+  <link name="front_bumper_mount"></link>
+  <joint name="front_bumper_mount_joint" type="fixed">
+    <origin xyz="0.275 0 0.04" rpy="0 0 0" />
+    <parent link="chassis_link"/>
+    <child link="front_bumper_mount" />
+  </joint>
+  <link name="rear_bumper_mount"></link>
+  <joint name="rear_bumper_mount_joint" type="fixed">
+    <origin xyz="-0.275 0 0.04" rpy="0 0 ${PI}" />
+    <parent link="chassis_link"/>
+    <child link="rear_bumper_mount" />
   </joint>
   <!-- Bring in simulation data for Gazebo. -->

File: dingo_description/urdf/dingo-o.urdf.xacro (robot description, xacro)
@@ -107,9 +107,42 @@
     <child link="imu_link" />
   </joint>
+  <!--
+    Mounting points for accessories in the top channel.
+    These are flush with the top of the robot and all oriented to face forwards
+  -->
   <link name="front_mount"></link>
   <joint name="front_mount_joint" type="fixed">
-    <origin xyz="0.2 0 0.05" rpy="0 0 0" />
+    <origin xyz="0.28 0 0.068" rpy="0 0 0" />
     <parent link="chassis_link"/>
     <child link="front_mount" />
+  </joint>
+  <link name="mid_mount"></link>
+  <joint name="mid_mount_joint" type="fixed">
+    <origin xyz="0 0 0.067" rpy="0 0 0" />
+    <parent link="chassis_link"/>
+    <child link="mid_mount" />
+  </joint>
+  <link name="rear_mount"></link>
+  <joint name="rear_mount_joint" type="fixed">
+    <origin xyz="-0.28 0 0.068" rpy="0 0 0" />
+    <parent link="chassis_link"/>
+    <child link="rear_mount" />
+  </joint>
+  <!--
+    Mounting points for accessories on the front/rear bumpers.
+    Use with caution, but thin sensors (e.g Raspberry Pi NoIR camera) could
+    be mounted here for low-budget, front/rear-facing capabilities
+  -->
+  <link name="front_bumper_mount"></link>
+  <joint name="front_bumper_mount_joint" type="fixed">
+    <origin xyz="0.343 0 0.04" rpy="0 0 0" />
+    <parent link="chassis_link"/>
+    <child link="front_bumper_mount" />
+  </joint>
+  <link name="rear_bumper_mount"></link>
+  <joint name="rear_bumper_mount_joint" type="fixed">
+    <origin xyz="-0.343 0 0.04" rpy="0 0 ${PI}" />
+    <parent link="chassis_link"/>
+    <child link="rear_bumper_mount" />
   </joint>
   <!-- Bring in simulation data for Gazebo. -->

Commit message: Fix the measurements.  Keep the front/rear mounts 5cm back from the bumpers, move the bumper mounts to the center of the bumper

File: dingo_description/urdf/dingo-d.urdf.xacro (robot description, xacro)
@@ -162,5 +162,5 @@
   <link name="front_mount"></link>
   <joint name="front_mount_joint" type="fixed">
-    <origin xyz="0.2 0 0.068" rpy="0 0 0" />
+    <origin xyz="0.224 0 0.064263" rpy="0 0 0" />
     <parent link="chassis_link"/>
     <child link="front_mount" />
@@ -168,5 +168,5 @@
   <link name="mid_mount"></link>
   <joint name="mid_mount_joint" type="fixed">
-    <origin xyz="0 0 0.067" rpy="0 0 0" />
+    <origin xyz="0 0 0.064263" rpy="0 0 0" />
     <parent link="chassis_link"/>
     <child link="mid_mount" />
@@ -174,5 +174,5 @@
   <link name="rear_mount"></link>
   <joint name="rear_mount_joint" type="fixed">
-    <origin xyz="-0.2 0 0.068" rpy="0 0 0" />
+    <origin xyz="-0.224 0 0.064263" rpy="0 0 0" />
     <parent link="chassis_link"/>
     <child link="rear_mount" />
@@ -185,5 +185,5 @@
   <link name="front_bumper_mount"></link>
   <joint name="front_bumper_mount_joint" type="fixed">
-    <origin xyz="0.275 0 0.04" rpy="0 0 0" />
+    <origin xyz="0.274 0 0.0345125" rpy="0 0 0" />
     <parent link="chassis_link"/>
     <child link="front_bumper_mount" />
@@ -191,5 +191,5 @@
   <link name="rear_bumper_mount"></link>
   <joint name="rear_bumper_mount_joint" type="fixed">
-    <origin xyz="-0.275 0 0.04" rpy="0 0 ${PI}" />
+    <origin xyz="-0.274 0 0.0345125" rpy="0 0 ${PI}" />
     <parent link="chassis_link"/>
     <child link="rear_bumper_mount" />

File: dingo_description/urdf/dingo-o.urdf.xacro (robot description, xacro)
@@ -113,5 +113,5 @@
   <link name="front_mount"></link>
   <joint name="front_mount_joint" type="fixed">
-    <origin xyz="0.28 0 0.068" rpy="0 0 0" />
+    <origin xyz="0.29159 0 0.069023" rpy="0 0 0" />
     <parent link="chassis_link"/>
     <child link="front_mount" />
@@ -119,5 +119,5 @@
   <link name="mid_mount"></link>
   <joint name="mid_mount_joint" type="fixed">
-    <origin xyz="0 0 0.067" rpy="0 0 0" />
+    <origin xyz="0 0 0.069023" rpy="0 0 0" />
     <parent link="chassis_link"/>
     <child link="mid_mount" />
@@ -125,5 +125,5 @@
   <link name="rear_mount"></link>
   <joint name="rear_mount_joint" type="fixed">
-    <origin xyz="-0.28 0 0.068" rpy="0 0 0" />
+    <origin xyz="-0.29159 0 0.069023" rpy="0 0 0" />
     <parent link="chassis_link"/>
     <child link="rear_mount" />
@@ -136,5 +136,5 @@
   <link name="front_bumper_mount"></link>
   <joint name="front_bumper_mount_joint" type="fixed">
-    <origin xyz="0.343 0 0.04" rpy="0 0 0" />
+    <origin xyz="0.34159 0 0.0345115" rpy="0 0 0" />
     <parent link="chassis_link"/>
     <child link="front_bumper_mount" />
@@ -142,5 +142,5 @@
   <link name="rear_bumper_mount"></link>
   <joint name="rear_bumper_mount_joint" type="fixed">
-    <origin xyz="-0.343 0 0.04" rpy="0 0 ${PI}" />
+    <origin xyz="-0.34159 0 0.0345115" rpy="0 0 ${PI}" />
     <parent link="chassis_link"/>
     <child link="rear_bumper_mount" />

Commit message: Remove the rear_bumper_mount since that's where the HMI is, which would prevent anything from being reasonably mounted there

File: dingo_description/urdf/dingo-d.urdf.xacro (robot description, xacro)
@@ -179,7 +179,7 @@
   </joint>
   <!--
-    Mounting points for accessories on the front/rear bumpers.
+    Mounting point for accessories on the front bumper.
     Use with caution, but thin sensors (e.g Raspberry Pi NoIR camera) could
-    be mounted here for low-budget, front/rear-facing capabilities
+    be mounted here for low-budget, front-facing capabilities
   -->
   <link name="front_bumper_mount"></link>
@@ -188,10 +188,4 @@
     <parent link="chassis_link"/>
     <child link="front_bumper_mount" />
-  </joint>
-  <link name="rear_bumper_mount"></link>
-  <joint name="rear_bumper_mount_joint" type="fixed">
-    <origin xyz="-0.274 0 0.0345125" rpy="0 0 ${PI}" />
-    <parent link="chassis_link"/>
-    <child link="rear_bumper_mount" />
   </joint>
   <!-- Bring in simulation data for Gazebo. -->

File: dingo_description/urdf/dingo-o.urdf.xacro (robot description, xacro)
@@ -130,5 +130,5 @@
   </joint>
   <!--
-    Mounting points for accessories on the front/rear bumpers.
+    Mounting point for accessories on the front bumper.
     Use with caution, but thin sensors (e.g Raspberry Pi NoIR camera) could
     be mounted here for low-budget, front/rear-facing capabilities
@@ -139,10 +139,4 @@
     <parent link="chassis_link"/>
     <child link="front_bumper_mount" />
-  </joint>
-  <link name="rear_bumper_mount"></link>
-  <joint name="rear_bumper_mount_joint" type="fixed">
-    <origin xyz="-0.34159 0 0.0345115" rpy="0 0 ${PI}" />
-    <parent link="chassis_link"/>
-    <child link="rear_bumper_mount" />
   </joint>
   <!-- Bring in simulation data for Gazebo. -->

Commit message: Fix the mount links for Dingo-D and Dingo-O; -D doesn't technically have a mid_mount

File: dingo_description/urdf/dingo-d.urdf.xacro (robot description, xacro)
@@ -158,22 +158,48 @@
   <!--
     Mounting points for accessories in the top channel.
-    These are flush with the top of the robot and all oriented to face forwards
+    These are flush with the top of the robot and all oriented to face forwards.
+    Dingo-D has 6 evenly-spaced 80mm mounts
+    We name the mounts (from front to back)
+      - front
+      - front b
+      - front c
+      - rear c
+      - rear b
+      - rear
   -->
-  <link name="front_mount"></link>
+  <link name="front_mount"/>
+  <link name="front_b_mount"/>
+  <link name="front_c_mount"/>
+  <link name="rear_mount"/>
+  <link name="rear_b_mount"/>
+  <link name="rear_c_mount"/>
+  <joint name="front_c_mount_joint" type="fixed">
+    <origin xyz="0.040 0 0.064263" rpy="0 0 0" />
+    <parent link="chassis_link"/>
+    <child link="front_c_mount" />
+  </joint>
+  <joint name="front_b_mount_joint" type="fixed">
+    <origin xyz="0.080 0 0" rpy="0 0 0" />
+    <parent link="front_c_mount"/>
+    <child link="front_b_mount" />
+  </joint>
   <joint name="front_mount_joint" type="fixed">
-    <origin xyz="0.224 0 0.064263" rpy="0 0 0" />
-    <parent link="chassis_link"/>
+    <origin xyz="0.080 0 0" rpy="0 0 0" />
+    <parent link="front_b_mount"/>
     <child link="front_mount" />
   </joint>
-  <link name="mid_mount"></link>
-  <joint name="mid_mount_joint" type="fixed">
-    <origin xyz="0 0 0.064263" rpy="0 0 0" />
-    <parent link="chassis_link"/>
-    <child link="mid_mount" />
-  </joint>
-  <link name="rear_mount"></link>
-  <joint name="rear_mount_joint" type="fixed">
-    <origin xyz="-0.224 0 0.064263" rpy="0 0 0" />
-    <parent link="chassis_link"/>
+  <joint name="rear_c_mount_joint" type="fixed">
+    <origin xyz="-0.040 0 0.064263" rpy="0 0 0" />
+    <parent link="chassis_link"/>
+    <child link="rear_c_mount" />
+  </joint>
+  <joint name="rear_b_mount_joint" type="fixed">
+    <origin xyz="-0.080 0 0" rpy="0 0 0" />
+    <parent link="rear_c_mount"/>
+    <child link="rear_b_mount" />
+  </joint>
+  <joint name="rear_moint_joint" type="fixed">
+    <origin xyz="-0.080 0 0" rpy="0 0 0" />
+    <parent link="rear_b_mount"/>
     <child link="rear_mount" />
   </joint>

File: dingo_description/urdf/dingo-o.urdf.xacro (robot description, xacro)
@@ -109,13 +109,22 @@
   <!--
     Mounting points for accessories in the top channel.
-    These are flush with the top of the robot and all oriented to face forwards
+    These are flush with the top of the robot and all oriented to face forwards.
+    Dingo-D has 6 evenly-spaced 80mm mounts
+    We name the mounts (from front to back)
+      - front
+      - front b
+      - front c
+      - mid
+      - rear c
+      - rear b
+      - rear
   -->
-  <link name="front_mount"></link>
-  <joint name="front_mount_joint" type="fixed">
-    <origin xyz="0.29159 0 0.069023" rpy="0 0 0" />
-    <parent link="chassis_link"/>
-    <child link="front_mount" />
-  </joint>
-  <link name="mid_mount"></link>
+  <link name="front_mount"/>
+  <link name="front_b_mount"/>
+  <link name="front_c_mount"/>
+  <link name="rear_mount"/>
+  <link name="rear_b_mount"/>
+  <link name="rear_c_mount"/>
+  <link name="mid_mount"/>
   <joint name="mid_mount_joint" type="fixed">
     <origin xyz="0 0 0.069023" rpy="0 0 0" />
@@ -123,8 +132,32 @@
     <child link="mid_mount" />
   </joint>
-  <link name="rear_mount"></link>
-  <joint name="rear_mount_joint" type="fixed">
-    <origin xyz="-0.29159 0 0.069023" rpy="0 0 0" />
-    <parent link="chassis_link"/>
+  <joint name="front_c_mount_joint" type="fixed">
+    <origin xyz="0.080 0 0" rpy="0 0 0" />
+    <parent link="mid_mount"/>
+    <child link="front_c_mount" />
+  </joint>
+  <joint name="front_b_mount_joint" type="fixed">
+    <origin xyz="0.080 0 0" rpy="0 0 0" />
+    <parent link="front_c_mount"/>
+    <child link="front_b_mount" />
+  </joint>
+  <joint name="front_mount_joint" type="fixed">
+    <origin xyz="0.080 0 0" rpy="0 0 0" />
+    <parent link="front_b_mount"/>
+    <child link="front_mount" />
+  </joint>
+  <joint name="rear_c_mount_joint" type="fixed">
+    <origin xyz="-0.080 0 0" rpy="0 0 0" />
+    <parent link="mid_mount"/>
+    <child link="rear_c_mount" />
+  </joint>
+  <joint name="rear_b_mount_joint" type="fixed">
+    <origin xyz="-0.080 0 0" rpy="0 0 0" />
+    <parent link="rear_c_mount"/>
+    <child link="rear_b_mount" />
+  </joint>
+  <joint name="rear_moint_joint" type="fixed">
+    <origin xyz="-0.080 0 0" rpy="0 0 0" />
+    <parent link="rear_b_mount"/>
     <child link="rear_mount" />
   </joint>

Commit message: set use_sim_time for ros2_control to true

File: dingo_description/urdf/dingo-d.urdf.xacro (robot description, xacro)
@@ -2,5 +2,7 @@
 <robot name="dingo" xmlns:xacro="http://www.ros.org/wiki/xacro">
 	<!-- Enable setting arguments from the launch file -->
-  <xacro:arg name="physical_robot" default="true" />
+  <xacro:arg name="physical_robot" default="true"/>
+	<xacro:property name="control_empty_default" value="" />
+	<xacro:arg name="control_yaml_file" default="$(control_empty_default)"/>
   <xacro:property name="PI" value="3.1415926535897931" />
   <xacro:property name="wheel_radius" value="0.049" />

Commit message: Added PACS

File: dingo_description/urdf/dingo-d.urdf.xacro (robot description, xacro)
@@ -1,4 +1,5 @@
 <?xml version="1.0"?>
 <robot name="dingo" xmlns:xacro="http://www.ros.org/wiki/xacro">
+  <xacro:property name="pacs_enabled" value="$(optenv DINGO_PACS 0)"/>
   <xacro:property name="PI" value="3.1415926535897931" />
   <xacro:property name="wheel_radius" value="0.049" />
@@ -168,40 +169,42 @@
       - rear
   -->
-  <link name="front_mount"/>
-  <link name="front_b_mount"/>
-  <link name="front_c_mount"/>
-  <link name="rear_mount"/>
-  <link name="rear_b_mount"/>
-  <link name="rear_c_mount"/>
-  <joint name="front_c_mount_joint" type="fixed">
-    <origin xyz="0.040 0 0.064263" rpy="0 0 0" />
-    <parent link="chassis_link"/>
-    <child link="front_c_mount" />
-  </joint>
-  <joint name="front_b_mount_joint" type="fixed">
-    <origin xyz="0.080 0 0" rpy="0 0 0" />
-    <parent link="front_c_mount"/>
-    <child link="front_b_mount" />
-  </joint>
-  <joint name="front_mount_joint" type="fixed">
-    <origin xyz="0.080 0 0" rpy="0 0 0" />
-    <parent link="front_b_mount"/>
-    <child link="front_mount" />
-  </joint>
-  <joint name="rear_c_mount_joint" type="fixed">
-    <origin xyz="-0.040 0 0.064263" rpy="0 0 0" />
-    <parent link="chassis_link"/>
-    <child link="rear_c_mount" />
-  </joint>
-  <joint name="rear_b_mount_joint" type="fixed">
-    <origin xyz="-0.080 0 0" rpy="0 0 0" />
-    <parent link="rear_c_mount"/>
-    <child link="rear_b_mount" />
-  </joint>
-  <joint name="rear_moint_joint" type="fixed">
-    <origin xyz="-0.080 0 0" rpy="0 0 0" />
-    <parent link="rear_b_mount"/>
-    <child link="rear_mount" />
-  </joint>
+  <xacro:unless value="${pacs_enabled}">
+    <link name="front_mount"/>
+    <link name="front_b_mount"/>
+    <link name="front_c_mount"/>
+    <link name="rear_mount"/>
+    <link name="rear_b_mount"/>
+    <link name="rear_c_mount"/>
+    <joint name="front_c_mount_joint" type="fixed">
+      <origin xyz="0.040 0 0.064263" rpy="0 0 0" />
+      <parent link="chassis_link"/>
+      <child link="front_c_mount" />
+    </joint>
+    <joint name="front_b_mount_joint" type="fixed">
+      <origin xyz="0.080 0 0" rpy="0 0 0" />
+      <parent link="front_c_mount"/>
+      <child link="front_b_mount" />
+    </joint>
+    <joint name="front_mount_joint" type="fixed">
+      <origin xyz="0.080 0 0" rpy="0 0 0" />
+      <parent link="front_b_mount"/>
+      <child link="front_mount" />
+    </joint>
+    <joint name="rear_c_mount_joint" type="fixed">
+      <origin xyz="-0.040 0 0.064263" rpy="0 0 0" />
+      <parent link="chassis_link"/>
+      <child link="rear_c_mount" />
+    </joint>
+    <joint name="rear_b_mount_joint" type="fixed">
+      <origin xyz="-0.080 0 0" rpy="0 0 0" />
+      <parent link="rear_c_mount"/>
+      <child link="rear_b_mount" />
+    </joint>
+    <joint name="rear_moint_joint" type="fixed">
+      <origin xyz="-0.080 0 0" rpy="0 0 0" />
+      <parent link="rear_b_mount"/>
+      <child link="rear_mount" />
+    </joint>
+  </xacro:unless>
   <!--
     Mounting point for accessories on the front bumper.
@@ -215,4 +218,7 @@
     <child link="front_bumper_mount" />
   </joint>
+  <!-- PACS -->
+  <xacro:include filename="$(find dingo_description)/urdf/pacs.urdf.xacro"/>
+  <xacro:pacs/>
   <!-- Bring in simulation data for Gazebo. -->
   <xacro:include filename="$(find dingo_description)/urdf/dingo.gazebo" />

File: dingo_description/urdf/dingo-o.urdf.xacro (robot description, xacro)
@@ -1,4 +1,5 @@
 <?xml version="1.0"?>
 <robot name="dingo" xmlns:xacro="http://www.ros.org/wiki/xacro">
+  <xacro:property name="pacs_enabled" value="$(optenv DINGO_PACS 0)" />
   <xacro:property name="PI" value="3.1415926535897931" />
   <xacro:property name="wheelbase" value="0.570" />
@@ -120,46 +121,48 @@
       - rear
   -->
-  <link name="front_mount"/>
-  <link name="front_b_mount"/>
-  <link name="front_c_mount"/>
-  <link name="rear_mount"/>
-  <link name="rear_b_mount"/>
-  <link name="rear_c_mount"/>
-  <link name="mid_mount"/>
-  <joint name="mid_mount_joint" type="fixed">
-    <origin xyz="0 0 0.069023" rpy="0 0 0" />
-    <parent link="chassis_link"/>
-    <child link="mid_mount" />
-  </joint>
-  <joint name="front_c_mount_joint" type="fixed">
-    <origin xyz="0.080 0 0" rpy="0 0 0" />
-    <parent link="mid_mount"/>
-    <child link="front_c_mount" />
-  </joint>
-  <joint name="front_b_mount_joint" type="fixed">
-    <origin xyz="0.080 0 0" rpy="0 0 0" />
-    <parent link="front_c_mount"/>
-    <child link="front_b_mount" />
-  </joint>
-  <joint name="front_mount_joint" type="fixed">
-    <origin xyz="0.080 0 0" rpy="0 0 0" />
-    <parent link="front_b_mount"/>
-    <child link="front_mount" />
-  </joint>
-  <joint name="rear_c_mount_joint" type="fixed">
-    <origin xyz="-0.080 0 0" rpy="0 0 0" />
-    <parent link="mid_mount"/>
-    <child link="rear_c_mount" />
-  </joint>
-  <joint name="rear_b_mount_joint" type="fixed">
-    <origin xyz="-0.080 0 0" rpy="0 0 0" />
-    <parent link="rear_c_mount"/>
-    <child link="rear_b_mount" />
-  </joint>
-  <joint name="rear_moint_joint" type="fixed">
-    <origin xyz="-0.080 0 0" rpy="0 0 0" />
-    <parent link="rear_b_mount"/>
-    <child link="rear_mount" />
-  </joint>
+  <xacro:unless value="${pacs_enabled}">
+    <link name="front_mount"/>
+    <link name="front_b_mount"/>
+    <link name="front_c_mount"/>
+    <link name="rear_mount"/>
+    <link name="rear_b_mount"/>
+    <link name="rear_c_mount"/>
+    <link name="mid_mount"/>
+    <joint name="mid_mount_joint" type="fixed">
+      <origin xyz="0 0 0.069023" rpy="0 0 0" />
+      <parent link="chassis_link"/>
+      <child link="mid_mount" />
+    </joint>
+    <joint name="front_c_mount_joint" type="fixed">
+      <origin xyz="0.080 0 0" rpy="0 0 0" />
+      <parent link="mid_mount"/>
+      <child link="front_c_mount" />
+    </joint>
+    <joint name="front_b_mount_joint" type="fixed">
+      <origin xyz="0.080 0 0" rpy="0 0 0" />
+      <parent link="front_c_mount"/>
+      <child link="front_b_mount" />
+    </joint>
+    <joint name="front_mount_joint" type="fixed">
+      <origin xyz="0.080 0 0" rpy="0 0 0" />
+      <parent link="front_b_mount"/>
+      <child link="front_mount" />
+    </joint>
+    <joint name="rear_c_mount_joint" type="fixed">
+      <origin xyz="-0.080 0 0" rpy="0 0 0" />
+      <parent link="mid_mount"/>
+      <child link="rear_c_mount" />
+    </joint>
+    <joint name="rear_b_mount_joint" type="fixed">
+      <origin xyz="-0.080 0 0" rpy="0 0 0" />
+      <parent link="rear_c_mount"/>
+      <child link="rear_b_mount" />
+    </joint>
+    <joint name="rear_moint_joint" type="fixed">
+      <origin xyz="-0.080 0 0" rpy="0 0 0" />
+      <parent link="rear_b_mount"/>
+      <child link="rear_mount" />
+    </joint>
+  </xacro:unless>
   <!--
     Mounting point for accessories on the front bumper.
@@ -173,4 +176,7 @@
     <child link="front_bumper_mount" />
   </joint>
+  <!-- PACS -->
+  <xacro:include filename="$(find dingo_description)/urdf/pacs.urdf.xacro"/>
+  <xacro:pacs/>
   <!-- Bring in simulation data for Gazebo. -->
   <xacro:include filename="$(find dingo_description)/urdf/dingo.gazebo" />

Commit message: Changed enable envvar name

File: dingo_description/urdf/dingo-d.urdf.xacro (robot description, xacro)
@@ -1,5 +1,5 @@
 <?xml version="1.0"?>
 <robot name="dingo" xmlns:xacro="http://www.ros.org/wiki/xacro">
-  <xacro:property name="pacs_enabled" value="$(optenv DINGO_PACS 0)"/>
+  <xacro:property name="pacs_enabled" value="$(optenv DINGO_PACS_ENABLED 0)"/>
   <xacro:property name="PI" value="3.1415926535897931" />
   <xacro:property name="wheel_radius" value="0.049" />

File: dingo_description/urdf/dingo-o.urdf.xacro (robot description, xacro)
@@ -1,5 +1,5 @@
 <?xml version="1.0"?>
 <robot name="dingo" xmlns:xacro="http://www.ros.org/wiki/xacro">
-  <xacro:property name="pacs_enabled" value="$(optenv DINGO_PACS 0)" />
+  <xacro:property name="pacs_enabled" value="$(optenv DINGO_PACS_ENABLED 0)" />
   <xacro:property name="PI" value="3.1415926535897931" />
   <xacro:property name="wheelbase" value="0.570" />

File: dingo_description/urdf/pacs.urdf.xacro (robot description, xacro)
@@ -278,5 +278,5 @@
     <xacro:property name="omni" value="$(optenv DINGO_OMNI 0)"/>
     <xacro:property name="riser" value="$(optenv DINGO_PACS_RISER 0)"/>
-    <xacro:property name="pacs_enabled" value="$(optenv DINGO_PACS 1)" />
+    <xacro:property name="pacs_enabled" value="$(optenv DINGO_PACS_ENABLED 1)" />
     <xacro:if value="${pacs_enabled}">
       <xacro:property name="riser_x" value="0.0"/>
