Commit message: Fix the spawn position of the Hokuyo lidar & its focal point. Add the STLs for the LMS-1xx & Hokuyo lidars.  Add lms1xx as a dependency so that the lidar macro is available.

File: dingo_description/urdf/accessories.urdf.xacro (robot description, xacro)
@@ -16,5 +16,5 @@
                           topic="$(optenv DINGO_LASER_TOPIC front/scan)" />
       <joint name="$(optenv DINGO_LASER_MOUNT front)_laser_mount_joint" type="fixed">
-        <origin xyz="$(optenv DINGO_LASER_OFFSET 0.11 0 0)"
+        <origin xyz="$(optenv DINGO_LASER_OFFSET 0 0 0)"
                 rpy="$(optenv DINGO_LASER_RPY 0 0 0)" />
         <parent link="$(optenv DINGO_LASER_MOUNT front)_mount" />

File: dingo_description/urdf/accessories/hokuyo_ust10.urdf.xacro (robot description, xacro)
@@ -60,5 +60,5 @@
     <joint name="${prefix}_laser_joint" type="fixed">
       <!-- This offset is from the base of the bracket to the LIDAR's focal point. -->
-      <origin xyz="0 0 0.149" rpy="0 0 0" />
+      <origin xyz="0 0 0.055" rpy="0 0 0" />
       <parent link="${prefix}_laser_mount" />
       <child link="${prefix}_laser" />

Commit message: Start adding support for the Intel RealSense cameras as out-of-the-box accessories

File: dingo_description/urdf/accessories.urdf.xacro (robot description, xacro)
@@ -34,3 +34,100 @@
     </xacro:unless>
   </xacro:if>
+  <xacro:if value="$(optenv DINGO_REALSENSE 0)">
+    <xacro:property name="rs_model" value="$(optenv DINGO_REALSENSE_MODEL d435)" />
+    <xacro:if value="${rs_model == 'd435'}">
+      <xacro:include filename="$(find realsense2_description)/urdf/_d435.urdf.xacro" />
+      <xacro:sensor_d435 parent="$(optenv DINGO_REALSENSE_MOUNT front)_mount"
+                         name="$(optenv DINGO_REALSENSE_MOUNT front)_realsense">
+        <origin xyz="$(optenv DINGO_REALSENSE_OFFSET 0 0 0)" rpy="$(optenv DINGO_REALSENSE_RPY 0 0 0)" />
+      </xacro:sensor_d435>
+      <include filename="$(find dingo_description)/urdf/accessories/intel_realsense.urdf.xacro" />
+      <xacro:realsense_gazebo
+        prefix="$(optenv DINGO_REALSENSE_MOUNT front)"
+        frame="$(optenv DINGO_REALSENSE_MOUNT front)_realsense_link"
+        topic="$(optenv DINGO_REALSENSE_TOPIC realsense)"
+        h_fov="1.5184351666666667"
+        v_fov="1.0122901111111111"
+        min_range="0.105"
+        max_range="8.0"
+        width="640"
+        height="480"
+        update_rate="30" />
+    </xacro:if>
+    <xacro:if value="${rs_model == 'd435i'}">
+      <xacro:include filename="$(find realsense2_description)/urdf/_d435i.urdf.xacro" />
+      <xacro:sensor_d435i parent="$(optenv DINGO_REALSENSE_MOUNT front)_mount"
+                         name="$(optenv DINGO_REALSENSE_MOUNT front)_realsense">
+        <origin xyz="$(optenv DINGO_REALSENSE_OFFSET 0 0 0)" rpy="$(optenv DINGO_REALSENSE_RPY 0 0 0)" />
+      </xacro:sensor_d435i>
+      <include filename="$(find dingo_description)/urdf/accessories/intel_realsense.urdf.xacro" />
+      <xacro:realsense_gazebo
+        prefix="$(optenv DINGO_REALSENSE_MOUNT front)"
+        frame="$(optenv DINGO_REALSENSE_MOUNT front)_realsense_link"
+        topic="$(optenv DINGO_REALSENSE_TOPIC realsense)"
+        h_fov="1.5184351666666667"
+        v_fov="1.0122901111111111"
+        min_range="0.105"
+        max_range="8.0"
+        width="640"
+        height="480"
+        update_rate="30" />
+      <!--
+        Add the IMU plugin
+        The realsense2_camera driver splits the accelerometer and gyroscope data
+        across 2 topics: accel and gyro
+      -->
+      <gazebo>
+        <plugin name="d435_accel" filename="libhector_gazebo_ros_imu.so">
+          <robotNamespace>/</robotNamespace>
+          <updateRate>30.0</updateRate>
+          <bodyName>$(optenv DINGO_REALSENSE_MOUNT front)_realsense_link</bodyName>
+          <topicName>$(optenv DINGO_REALSENSE_TOPIC realsense)/accel/sample</topicName>
+          <accelDrift>0.005 0.005 0.005</accelDrift>
+          <accelGaussianNoise>0.005 0.005 0.005</accelGaussianNoise>
+          <rateDrift>0.005 0.005 0.005 </rateDrift>
+          <rateGaussianNoise>0.005 0.005 0.005 </rateGaussianNoise>
+          <headingDrift>0.005</headingDrift>
+          <headingGaussianNoise>0.005</headingGaussianNoise>
+        </plugin>
+        <plugin name="d435_gyro" filename="libhector_gazebo_ros_imu.so">
+          <robotNamespace>/</robotNamespace>
+          <updateRate>30.0</updateRate>
+          <bodyName>$(optenv DINGO_REALSENSE_MOUNT front)_realsense_link</bodyName>
+          <topicName>$(optenv DINGO_REALSENSE_TOPIC realsense)/gyro/sample</topicName>
+          <accelDrift>0.005 0.005 0.005</accelDrift>
+          <accelGaussianNoise>0.005 0.005 0.005</accelGaussianNoise>
+          <rateDrift>0.005 0.005 0.005 </rateDrift>
+          <rateGaussianNoise>0.005 0.005 0.005 </rateGaussianNoise>
+          <headingDrift>0.005</headingDrift>
+          <headingGaussianNoise>0.005</headingGaussianNoise>
+        </plugin>
+      </gazebo>
+    </xacro:if>
+    <xacro:if value="${rs_model == 'd415'}">
+      <xacro:include filename="$(find realsense2_description)/urdf/_d415.urdf.xacro" />
+      <xacro:sensor_d415 parent="$(optenv DINGO_REALSENSE_MOUNT front)_mount"
+                         name="$(optenv DINGO_REALSENSE_MOUNT front)_realsense">
+        <origin xyz="$(optenv DINGO_REALSENSE_OFFSET 0 0 0)" rpy="$(optenv DINGO_REALSENSE_RPY 0 0 0)" />
+      </xacro:sensor_d415>
+      <include filename="$(find dingo_description)/urdf/accessories/intel_realsense.urdf.xacro" />
+      <xacro:realsense_gazebo
+        prefix="$(optenv DINGO_REALSENSE_MOUNT front)"
+        frame="$(optenv DINGO_REALSENSE_MOUNT front)_realsense_link"
+        topic="$(optenv DINGO_REALSENSE_TOPIC realsense)"
+        h_fov="1.1344640137963142"
+        v_fov="0.6981317007977318"
+        min_range="0.3"
+        max_range="5.0"
+        width="640"
+        height="480"
+        update_rate="30" />
+    </xacro:if>
+    <xacro:if value="${rs_model == 'd455'}">
+      <!-- TODO: not officially supported yet -->
+    </xacro:if>
+    <xacro:if value="${rs_model == 'l515'}">
+      <!-- TODO: not officially supported yet -->
+    </xacro:if>
+  </xacro:if>
 </robot>

Commit message: Refactor the lidar accessory variables, add clarifying comments to make it easier to find supported values for the sensor models

File: dingo_description/urdf/accessories.urdf.xacro (robot description, xacro)
@@ -9,7 +9,24 @@
     dingo_base/launch/base.launch
   -->
-  <!-- If enabled, generate the LASER payload (by default, a SICK LMS111). -->
+  <!--
+    Add a lidar sensor.  By default this is a SICK LMS1xx but can be changed with the
+    DINGO_LASER_MODEL environment variable. Valid model designations are:
+    - lms1xx (default) :: SICK LMS1xx
+    - ust10            :: Hokuyo UST10
+  -->
   <xacro:if value="$(optenv DINGO_LASER 0)">
-    <xacro:if value="$(optenv DINGO_LASER_HOKUYO 0)">
+    <xacro:property name="lidar_model" value="$(optenv DINGO_LASER_MODEL lms1xx)" />
+    <xacro:if value="${lidar_model == lms1xx}">
+      <xacro:include filename="$(find dingo_description)/urdf/accessories/sick_lms1xx_mount.urdf.xacro" />
+      <xacro:sick_lms1xx_mount prefix="$(optenv DINGO_LASER_MOUNT front)"
+                         topic="$(optenv DINGO_LASER_TOPIC front/scan)"/>
+      <joint name="$(optenv DINGO_LASER_MOUNT front)_laser_mount_joint" type="fixed">
+        <origin xyz="$(optenv DINGO_LASER_OFFSET 0 0 0)"
+                rpy="$(optenv DINGO_LASER_RPY 0 0 0)" />
+        <parent link="$(optenv DINGO_LASER_MOUNT front)_mount" />
+        <child link="$(optenv DINGO_LASER_MOUNT front)_laser_mount" />
+      </joint>
+    </xacro:if>
+    <xacro:if value="${lidar_model == ust10}">
       <xacro:include filename="$(find dingo_description)/urdf/accessories/hokuyo_ust10.urdf.xacro" />
       <xacro:hokuyo_ust10_mount prefix="$(optenv DINGO_LASER_MOUNT front)"
@@ -22,16 +39,14 @@
       </joint>
     </xacro:if>
-    <xacro:unless value="$(optenv DINGO_LASER_HOKUYO 0)">
-      <xacro:include filename="$(find dingo_description)/urdf/accessories/sick_lms1xx_mount.urdf.xacro" />
-      <xacro:sick_lms1xx_mount prefix="$(optenv DINGO_LASER_MOUNT front)"
-                         topic="$(optenv DINGO_LASER_TOPIC front/scan)"/>
-      <joint name="$(optenv DINGO_LASER_MOUNT front)_laser_mount_joint" type="fixed">
-        <origin xyz="$(optenv DINGO_LASER_OFFSET 0 0 0)"
-                rpy="$(optenv DINGO_LASER_RPY 0 0 0)" />
-        <parent link="$(optenv DINGO_LASER_MOUNT front)_mount" />
-        <child link="$(optenv DINGO_LASER_MOUNT front)_laser_mount" />
-      </joint>
-    </xacro:unless>
   </xacro:if>
+  <!--
+    Add an Intel RealSense family camera.  By default this is a D435, but can be changed with the
+    DINGO_REALSENSE_MODEL environment variable. Valid model designations are:
+    - d435 (default)
+    - d435i
+    - d415
+    - d455
+    - l515
+  -->
   <xacro:if value="$(optenv DINGO_REALSENSE 0)">
     <xacro:property name="rs_model" value="$(optenv DINGO_REALSENSE_MODEL d435)" />

Commit message: Model Update (#3)
* Make the yellow of the chassis more yellow and less orange

* Fix the spawn position of the Hokuyo lidar & its focal point. Add the STLs for the LMS-1xx & Hokuyo lidars.  Add lms1xx as a dependency so that the lidar macro is available.

* Add additional mounting points for accessories, fix the position of the existing front_mount

* Start adding support for the Intel RealSense cameras as out-of-the-box accessories

* Update the dependencies

* Remove the hector gazebo plugin dependency; it's included in dingo_gazebo, and isn't strictly needed in the description package

* Refactor the lidar accessory variables, add clarifying comments to make it easier to find supported values for the sensor models

* Fix the measurements.  Keep the front/rear mounts 5cm back from the bumpers, move the bumper mounts to the center of the bumper

* Remove the rear_bumper_mount since that's where the HMI is, which would prevent anything from being reasonably mounted there

File: dingo_description/urdf/accessories.urdf.xacro (robot description, xacro)
@@ -9,7 +9,24 @@
     dingo_base/launch/base.launch
   -->
-  <!-- If enabled, generate the LASER payload (by default, a SICK LMS111). -->
+  <!--
+    Add a lidar sensor.  By default this is a SICK LMS1xx but can be changed with the
+    DINGO_LASER_MODEL environment variable. Valid model designations are:
+    - lms1xx (default) :: SICK LMS1xx
+    - ust10            :: Hokuyo UST10
+  -->
   <xacro:if value="$(optenv DINGO_LASER 0)">
-    <xacro:if value="$(optenv DINGO_LASER_HOKUYO 0)">
+    <xacro:property name="lidar_model" value="$(optenv DINGO_LASER_MODEL lms1xx)" />
+    <xacro:if value="${lidar_model == lms1xx}">
+      <xacro:include filename="$(find dingo_description)/urdf/accessories/sick_lms1xx_mount.urdf.xacro" />
+      <xacro:sick_lms1xx_mount prefix="$(optenv DINGO_LASER_MOUNT front)"
+                         topic="$(optenv DINGO_LASER_TOPIC front/scan)"/>
+      <joint name="$(optenv DINGO_LASER_MOUNT front)_laser_mount_joint" type="fixed">
+        <origin xyz="$(optenv DINGO_LASER_OFFSET 0 0 0)"
+                rpy="$(optenv DINGO_LASER_RPY 0 0 0)" />
+        <parent link="$(optenv DINGO_LASER_MOUNT front)_mount" />
+        <child link="$(optenv DINGO_LASER_MOUNT front)_laser_mount" />
+      </joint>
+    </xacro:if>
+    <xacro:if value="${lidar_model == ust10}">
       <xacro:include filename="$(find dingo_description)/urdf/accessories/hokuyo_ust10.urdf.xacro" />
       <xacro:hokuyo_ust10_mount prefix="$(optenv DINGO_LASER_MOUNT front)"
@@ -22,15 +39,110 @@
       </joint>
     </xacro:if>
-    <xacro:unless value="$(optenv DINGO_LASER_HOKUYO 0)">
-      <xacro:include filename="$(find dingo_description)/urdf/accessories/sick_lms1xx_mount.urdf.xacro" />
-      <xacro:sick_lms1xx_mount prefix="$(optenv DINGO_LASER_MOUNT front)"
-                         topic="$(optenv DINGO_LASER_TOPIC front/scan)"/>
-      <joint name="$(optenv DINGO_LASER_MOUNT front)_laser_mount_joint" type="fixed">
-        <origin xyz="$(optenv DINGO_LASER_OFFSET 0 0 0)"
-                rpy="$(optenv DINGO_LASER_RPY 0 0 0)" />
-        <parent link="$(optenv DINGO_LASER_MOUNT front)_mount" />
-        <child link="$(optenv DINGO_LASER_MOUNT front)_laser_mount" />
-      </joint>
-    </xacro:unless>
+  </xacro:if>
+  <!--
+    Add an Intel RealSense family camera.  By default this is a D435, but can be changed with the
+    DINGO_REALSENSE_MODEL environment variable. Valid model designations are:
+    - d435 (default)
+    - d435i
+    - d415
+    - d455
+    - l515
+  -->
+  <xacro:if value="$(optenv DINGO_REALSENSE 0)">
+    <xacro:property name="rs_model" value="$(optenv DINGO_REALSENSE_MODEL d435)" />
+    <xacro:if value="${rs_model == 'd435'}">
+      <xacro:include filename="$(find realsense2_description)/urdf/_d435.urdf.xacro" />
+      <xacro:sensor_d435 parent="$(optenv DINGO_REALSENSE_MOUNT front)_mount"
+                         name="$(optenv DINGO_REALSENSE_MOUNT front)_realsense">
+        <origin xyz="$(optenv DINGO_REALSENSE_OFFSET 0 0 0)" rpy="$(optenv DINGO_REALSENSE_RPY 0 0 0)" />
+      </xacro:sensor_d435>
+      <include filename="$(find dingo_description)/urdf/accessories/intel_realsense.urdf.xacro" />
+      <xacro:realsense_gazebo
+        prefix="$(optenv DINGO_REALSENSE_MOUNT front)"
+        frame="$(optenv DINGO_REALSENSE_MOUNT front)_realsense_link"
+        topic="$(optenv DINGO_REALSENSE_TOPIC realsense)"
+        h_fov="1.5184351666666667"
+        v_fov="1.0122901111111111"
+        min_range="0.105"
+        max_range="8.0"
+        width="640"
+        height="480"
+        update_rate="30" />
+    </xacro:if>
+    <xacro:if value="${rs_model == 'd435i'}">
+      <xacro:include filename="$(find realsense2_description)/urdf/_d435i.urdf.xacro" />
+      <xacro:sensor_d435i parent="$(optenv DINGO_REALSENSE_MOUNT front)_mount"
+                         name="$(optenv DINGO_REALSENSE_MOUNT front)_realsense">
+        <origin xyz="$(optenv DINGO_REALSENSE_OFFSET 0 0 0)" rpy="$(optenv DINGO_REALSENSE_RPY 0 0 0)" />
+      </xacro:sensor_d435i>
+      <include filename="$(find dingo_description)/urdf/accessories/intel_realsense.urdf.xacro" />
+      <xacro:realsense_gazebo
+        prefix="$(optenv DINGO_REALSENSE_MOUNT front)"
+        frame="$(optenv DINGO_REALSENSE_MOUNT front)_realsense_link"
+        topic="$(optenv DINGO_REALSENSE_TOPIC realsense)"
+        h_fov="1.5184351666666667"
+        v_fov="1.0122901111111111"
+        min_range="0.105"
+        max_range="8.0"
+        width="640"
+        height="480"
+        update_rate="30" />
+      <!--
+        Add the IMU plugin
+        The realsense2_camera driver splits the accelerometer and gyroscope data
+        across 2 topics: accel and gyro
+      -->
+      <gazebo>
+        <plugin name="d435_accel" filename="libhector_gazebo_ros_imu.so">
+          <robotNamespace>/</robotNamespace>
+          <updateRate>30.0</updateRate>
+          <bodyName>$(optenv DINGO_REALSENSE_MOUNT front)_realsense_link</bodyName>
+          <topicName>$(optenv DINGO_REALSENSE_TOPIC realsense)/accel/sample</topicName>
+          <accelDrift>0.005 0.005 0.005</accelDrift>
+          <accelGaussianNoise>0.005 0.005 0.005</accelGaussianNoise>
+          <rateDrift>0.005 0.005 0.005 </rateDrift>
+          <rateGaussianNoise>0.005 0.005 0.005 </rateGaussianNoise>
+          <headingDrift>0.005</headingDrift>
+          <headingGaussianNoise>0.005</headingGaussianNoise>
+        </plugin>
+        <plugin name="d435_gyro" filename="libhector_gazebo_ros_imu.so">
+          <robotNamespace>/</robotNamespace>
+          <updateRate>30.0</updateRate>
+          <bodyName>$(optenv DINGO_REALSENSE_MOUNT front)_realsense_link</bodyName>
+          <topicName>$(optenv DINGO_REALSENSE_TOPIC realsense)/gyro/sample</topicName>
+          <accelDrift>0.005 0.005 0.005</accelDrift>
+          <accelGaussianNoise>0.005 0.005 0.005</accelGaussianNoise>
+          <rateDrift>0.005 0.005 0.005 </rateDrift>
+          <rateGaussianNoise>0.005 0.005 0.005 </rateGaussianNoise>
+          <headingDrift>0.005</headingDrift>
+          <headingGaussianNoise>0.005</headingGaussianNoise>
+        </plugin>
+      </gazebo>
+    </xacro:if>
+    <xacro:if value="${rs_model == 'd415'}">
+      <xacro:include filename="$(find realsense2_description)/urdf/_d415.urdf.xacro" />
+      <xacro:sensor_d415 parent="$(optenv DINGO_REALSENSE_MOUNT front)_mount"
+                         name="$(optenv DINGO_REALSENSE_MOUNT front)_realsense">
+        <origin xyz="$(optenv DINGO_REALSENSE_OFFSET 0 0 0)" rpy="$(optenv DINGO_REALSENSE_RPY 0 0 0)" />
+      </xacro:sensor_d415>
+      <include filename="$(find dingo_description)/urdf/accessories/intel_realsense.urdf.xacro" />
+      <xacro:realsense_gazebo
+        prefix="$(optenv DINGO_REALSENSE_MOUNT front)"
+        frame="$(optenv DINGO_REALSENSE_MOUNT front)_realsense_link"
+        topic="$(optenv DINGO_REALSENSE_TOPIC realsense)"
+        h_fov="1.1344640137963142"
+        v_fov="0.6981317007977318"
+        min_range="0.3"
+        max_range="5.0"
+        width="640"
+        height="480"
+        update_rate="30" />
+    </xacro:if>
+    <xacro:if value="${rs_model == 'd455'}">
+      <!-- TODO: not officially supported yet -->
+    </xacro:if>
+    <xacro:if value="${rs_model == 'l515'}">
+      <!-- TODO: not officially supported yet -->
+    </xacro:if>
   </xacro:if>
 </robot>

File: dingo_description/urdf/dingo-d.urdf.xacro (robot description, xacro)
@@ -156,9 +156,36 @@
     <child link="imu_link" />
   </joint>
+  <!--
+    Mounting points for accessories in the top channel.
+    These are flush with the top of the robot and all oriented to face forwards
+  -->
   <link name="front_mount"></link>
   <joint name="front_mount_joint" type="fixed">
-    <origin xyz="0.2 0 0.05" rpy="0 0 0" />
+    <origin xyz="0.224 0 0.064263" rpy="0 0 0" />
     <parent link="chassis_link"/>
     <child link="front_mount" />
+  </joint>
+  <link name="mid_mount"></link>
+  <joint name="mid_mount_joint" type="fixed">
+    <origin xyz="0 0 0.064263" rpy="0 0 0" />
+    <parent link="chassis_link"/>
+    <child link="mid_mount" />
+  </joint>
+  <link name="rear_mount"></link>
+  <joint name="rear_mount_joint" type="fixed">
+    <origin xyz="-0.224 0 0.064263" rpy="0 0 0" />
+    <parent link="chassis_link"/>
+    <child link="rear_mount" />
+  </joint>
+  <!--
+    Mounting point for accessories on the front bumper.
+    Use with caution, but thin sensors (e.g Raspberry Pi NoIR camera) could
+    be mounted here for low-budget, front-facing capabilities
+  -->
+  <link name="front_bumper_mount"></link>
+  <joint name="front_bumper_mount_joint" type="fixed">
+    <origin xyz="0.274 0 0.0345125" rpy="0 0 0" />
+    <parent link="chassis_link"/>
+    <child link="front_bumper_mount" />
   </joint>
   <!-- Bring in simulation data for Gazebo. -->

File: dingo_description/urdf/dingo-o.urdf.xacro (robot description, xacro)
@@ -107,9 +107,36 @@
     <child link="imu_link" />
   </joint>
+  <!--
+    Mounting points for accessories in the top channel.
+    These are flush with the top of the robot and all oriented to face forwards
+  -->
   <link name="front_mount"></link>
   <joint name="front_mount_joint" type="fixed">
-    <origin xyz="0.2 0 0.05" rpy="0 0 0" />
+    <origin xyz="0.29159 0 0.069023" rpy="0 0 0" />
     <parent link="chassis_link"/>
     <child link="front_mount" />
+  </joint>
+  <link name="mid_mount"></link>
+  <joint name="mid_mount_joint" type="fixed">
+    <origin xyz="0 0 0.069023" rpy="0 0 0" />
+    <parent link="chassis_link"/>
+    <child link="mid_mount" />
+  </joint>
+  <link name="rear_mount"></link>
+  <joint name="rear_mount_joint" type="fixed">
+    <origin xyz="-0.29159 0 0.069023" rpy="0 0 0" />
+    <parent link="chassis_link"/>
+    <child link="rear_mount" />
+  </joint>
+  <!--
+    Mounting point for accessories on the front bumper.
+    Use with caution, but thin sensors (e.g Raspberry Pi NoIR camera) could
+    be mounted here for low-budget, front/rear-facing capabilities
+  -->
+  <link name="front_bumper_mount"></link>
+  <joint name="front_bumper_mount_joint" type="fixed">
+    <origin xyz="0.34159 0 0.0345115" rpy="0 0 0" />
+    <parent link="chassis_link"/>
+    <child link="front_bumper_mount" />
   </joint>
   <!-- Bring in simulation data for Gazebo. -->
