Commit message: Add placeholder support for the RS L515 and D455 so that the gazebo plugins work; the meshes for these sensors don't exist yet, but we can at least get the plugin configured & add the appropriate links for now

File: dingo_description/urdf/accessories.urdf.xacro (robot description, xacro)
@@ -140,8 +140,42 @@
     </xacro:if>
     <xacro:if value="${rs_model == 'd455'}">
-      <!-- TODO: not officially supported yet -->
+      <!-- TODO: not officially supported yet. Use the D435 mesh for now, even though it's the wrong size -->
+      <xacro:include filename="$(find realsense2_description)/urdf/_d435.urdf.xacro" />
+      <xacro:sensor_d435 parent="$(optenv DINGO_REALSENSE_MOUNT front)_mount"
+                         name="$(optenv DINGO_REALSENSE_MOUNT front)_realsense">
+        <origin xyz="$(optenv DINGO_REALSENSE_OFFSET 0 0 0)" rpy="$(optenv DINGO_REALSENSE_RPY 0 0 0)" />
+      </xacro:sensor_d435>
+      <include filename="$(find dingo_description)/urdf/accessories/intel_realsense.urdf.xacro" />
+      <xacro:realsense_gazebo
+        prefix="$(optenv DINGO_REALSENSE_MOUNT front)"
+        frame="$(optenv DINGO_REALSENSE_MOUNT front)_realsense_link"
+        topic="$(optenv DINGO_REALSENSE_TOPIC realsense)"
+        h_fov="1.5009831567151233"
+        v_fov="0.9948376736367678"
+        min_range="0.5"
+        max_range="20.0"
+        width="640"
+        height="480"
+        update_rate="30" />
     </xacro:if>
     <xacro:if value="${rs_model == 'l515'}">
-      <!-- TODO: not officially supported yet -->
+      <!-- TODO: not officially supported yet. Use the D435 mesh for now, even though it's the wrong shape -->
+      <xacro:include filename="$(find realsense2_description)/urdf/_d435.urdf.xacro" />
+      <xacro:sensor_d435 parent="$(optenv DINGO_REALSENSE_MOUNT front)_mount"
+                         name="$(optenv DINGO_REALSENSE_MOUNT front)_realsense">
+        <origin xyz="$(optenv DINGO_REALSENSE_OFFSET 0 0 0)" rpy="$(optenv DINGO_REALSENSE_RPY 0 0 0)" />
+      </xacro:sensor_d435>
+      <include filename="$(find dingo_description)/urdf/accessories/intel_realsense.urdf.xacro" />
+      <xacro:realsense_gazebo
+        prefix="$(optenv DINGO_REALSENSE_MOUNT front)"
+        frame="$(optenv DINGO_REALSENSE_MOUNT front)_realsense_link"
+        topic="$(optenv DINGO_REALSENSE_TOPIC realsense)"
+        h_fov="1.2217304763960306"
+        v_fov="0.9599310885968813"
+        min_range="0.25"
+        max_range="9.0"
+        width="640"
+        height="480"
+        update_rate="30" />
     </xacro:if>
   </xacro:if>
