Commit message: Refactor the RealSense macro to put the mesh + gazebo plugin in one place. Create a more-accurate L515 mesh out of cylinders until Intel releases an official mesh for the sensor

File: dingo_description/urdf/accessories.urdf.xacro (robot description, xacro)
@@ -50,133 +50,8 @@
   -->
   <xacro:if value="$(optenv DINGO_REALSENSE 0)">
-    <xacro:property name="rs_model" value="$(optenv DINGO_REALSENSE_MODEL d435)" />
-    <xacro:if value="${rs_model == 'd435'}">
-      <xacro:include filename="$(find realsense2_description)/urdf/_d435.urdf.xacro" />
-      <xacro:sensor_d435 parent="$(optenv DINGO_REALSENSE_MOUNT front)_mount"
-                         name="$(optenv DINGO_REALSENSE_MOUNT front)_realsense">
-        <origin xyz="$(optenv DINGO_REALSENSE_OFFSET 0 0 0)" rpy="$(optenv DINGO_REALSENSE_RPY 0 0 0)" />
-      </xacro:sensor_d435>
-      <include filename="$(find dingo_description)/urdf/accessories/intel_realsense.urdf.xacro" />
-      <xacro:realsense_gazebo
-        prefix="$(optenv DINGO_REALSENSE_MOUNT front)"
-        frame="$(optenv DINGO_REALSENSE_MOUNT front)_realsense_link"
-        topic="$(optenv DINGO_REALSENSE_TOPIC realsense)"
-        h_fov="1.5184351666666667"
-        v_fov="1.0122901111111111"
-        min_range="0.105"
-        max_range="8.0"
-        width="640"
-        height="480"
-        update_rate="30" />
-    </xacro:if>
-    <xacro:if value="${rs_model == 'd435i'}">
-      <xacro:include filename="$(find realsense2_description)/urdf/_d435i.urdf.xacro" />
-      <xacro:sensor_d435i parent="$(optenv DINGO_REALSENSE_MOUNT front)_mount"
-                         name="$(optenv DINGO_REALSENSE_MOUNT front)_realsense">
-        <origin xyz="$(optenv DINGO_REALSENSE_OFFSET 0 0 0)" rpy="$(optenv DINGO_REALSENSE_RPY 0 0 0)" />
-      </xacro:sensor_d435i>
-      <include filename="$(find dingo_description)/urdf/accessories/intel_realsense.urdf.xacro" />
-      <xacro:realsense_gazebo
-        prefix="$(optenv DINGO_REALSENSE_MOUNT front)"
-        frame="$(optenv DINGO_REALSENSE_MOUNT front)_realsense_link"
-        topic="$(optenv DINGO_REALSENSE_TOPIC realsense)"
-        h_fov="1.5184351666666667"
-        v_fov="1.0122901111111111"
-        min_range="0.105"
-        max_range="8.0"
-        width="640"
-        height="480"
-        update_rate="30" />
-      <!--
-        Add the IMU plugin
-        The realsense2_camera driver splits the accelerometer and gyroscope data
-        across 2 topics: accel and gyro
-      -->
-      <gazebo>
-        <plugin name="d435_accel" filename="libhector_gazebo_ros_imu.so">
-          <robotNamespace>/</robotNamespace>
-          <updateRate>30.0</updateRate>
-          <bodyName>$(optenv DINGO_REALSENSE_MOUNT front)_realsense_link</bodyName>
-          <topicName>$(optenv DINGO_REALSENSE_TOPIC realsense)/accel/sample</topicName>
-          <accelDrift>0.005 0.005 0.005</accelDrift>
-          <accelGaussianNoise>0.005 0.005 0.005</accelGaussianNoise>
-          <rateDrift>0.005 0.005 0.005 </rateDrift>
-          <rateGaussianNoise>0.005 0.005 0.005 </rateGaussianNoise>
-          <headingDrift>0.005</headingDrift>
-          <headingGaussianNoise>0.005</headingGaussianNoise>
-        </plugin>
-        <plugin name="d435_gyro" filename="libhector_gazebo_ros_imu.so">
-          <robotNamespace>/</robotNamespace>
-          <updateRate>30.0</updateRate>
-          <bodyName>$(optenv DINGO_REALSENSE_MOUNT front)_realsense_link</bodyName>
-          <topicName>$(optenv DINGO_REALSENSE_TOPIC realsense)/gyro/sample</topicName>
-          <accelDrift>0.005 0.005 0.005</accelDrift>
-          <accelGaussianNoise>0.005 0.005 0.005</accelGaussianNoise>
-          <rateDrift>0.005 0.005 0.005 </rateDrift>
-          <rateGaussianNoise>0.005 0.005 0.005 </rateGaussianNoise>
-          <headingDrift>0.005</headingDrift>
-          <headingGaussianNoise>0.005</headingGaussianNoise>
-        </plugin>
-      </gazebo>
-    </xacro:if>
-    <xacro:if value="${rs_model == 'd415'}">
-      <xacro:include filename="$(find realsense2_description)/urdf/_d415.urdf.xacro" />
-      <xacro:sensor_d415 parent="$(optenv DINGO_REALSENSE_MOUNT front)_mount"
-                         name="$(optenv DINGO_REALSENSE_MOUNT front)_realsense">
-        <origin xyz="$(optenv DINGO_REALSENSE_OFFSET 0 0 0)" rpy="$(optenv DINGO_REALSENSE_RPY 0 0 0)" />
-      </xacro:sensor_d415>
-      <include filename="$(find dingo_description)/urdf/accessories/intel_realsense.urdf.xacro" />
-      <xacro:realsense_gazebo
-        prefix="$(optenv DINGO_REALSENSE_MOUNT front)"
-        frame="$(optenv DINGO_REALSENSE_MOUNT front)_realsense_link"
-        topic="$(optenv DINGO_REALSENSE_TOPIC realsense)"
-        h_fov="1.1344640137963142"
-        v_fov="0.6981317007977318"
-        min_range="0.3"
-        max_range="5.0"
-        width="640"
-        height="480"
-        update_rate="30" />
-    </xacro:if>
-    <xacro:if value="${rs_model == 'd455'}">
-      <!-- TODO: not officially supported yet. Use the D435 mesh for now, even though it's the wrong size -->
-      <xacro:include filename="$(find realsense2_description)/urdf/_d435.urdf.xacro" />
-      <xacro:sensor_d435 parent="$(optenv DINGO_REALSENSE_MOUNT front)_mount"
-                         name="$(optenv DINGO_REALSENSE_MOUNT front)_realsense">
-        <origin xyz="$(optenv DINGO_REALSENSE_OFFSET 0 0 0)" rpy="$(optenv DINGO_REALSENSE_RPY 0 0 0)" />
-      </xacro:sensor_d435>
-      <include filename="$(find dingo_description)/urdf/accessories/intel_realsense.urdf.xacro" />
-      <xacro:realsense_gazebo
-        prefix="$(optenv DINGO_REALSENSE_MOUNT front)"
-        frame="$(optenv DINGO_REALSENSE_MOUNT front)_realsense_link"
-        topic="$(optenv DINGO_REALSENSE_TOPIC realsense)"
-        h_fov="1.5009831567151233"
-        v_fov="0.9948376736367678"
-        min_range="0.5"
-        max_range="20.0"
-        width="640"
-        height="480"
-        update_rate="30" />
-    </xacro:if>
-    <xacro:if value="${rs_model == 'l515'}">
-      <!-- TODO: not officially supported yet. Use the D435 mesh for now, even though it's the wrong shape -->
-      <xacro:include filename="$(find realsense2_description)/urdf/_d435.urdf.xacro" />
-      <xacro:sensor_d435 parent="$(optenv DINGO_REALSENSE_MOUNT front)_mount"
-                         name="$(optenv DINGO_REALSENSE_MOUNT front)_realsense">
-        <origin xyz="$(optenv DINGO_REALSENSE_OFFSET 0 0 0)" rpy="$(optenv DINGO_REALSENSE_RPY 0 0 0)" />
-      </xacro:sensor_d435>
-      <include filename="$(find dingo_description)/urdf/accessories/intel_realsense.urdf.xacro" />
-      <xacro:realsense_gazebo
-        prefix="$(optenv DINGO_REALSENSE_MOUNT front)"
-        frame="$(optenv DINGO_REALSENSE_MOUNT front)_realsense_link"
-        topic="$(optenv DINGO_REALSENSE_TOPIC realsense)"
-        h_fov="1.2217304763960306"
-        v_fov="0.9599310885968813"
-        min_range="0.25"
-        max_range="9.0"
-        width="640"
-        height="480"
-        update_rate="30" />
-    </xacro:if>
+    <include filename="$(find dingo_description)/urdf/accessories/intel_realsense.urdf.xacro" />
+    <xacro:realsense_sensor rs_model="$(optenv DINGO_REALSENSE_MODEL d435)"
+                            prefix="$(optenv DINGO_REALSENSE_MOUNT front)"
+                            topic="$(optenv DINGO_REALSENSE_TOPIC realsense)" />
   </xacro:if>
 </robot>

File: dingo_description/urdf/accessories/intel_realsense.urdf.xacro (robot description, xacro)
@@ -2,72 +2,233 @@
 <!--
   The realsense2_description package doesn't natively support simulation, so this
-  file defines a simple macro to use the kinect gazebo plugin to simulate data from the camera
+  file is a wrapper or the realsense2_description macro that also uses the kinect
+  gazebo plugin to simulate data from the camera
 -->
 <robot xmlns:xacro="http://ros.org/wiki/xacro">
-  <xacro:macro name="realsense_gazebo" params="
-             prefix=front
-             frame:=realsense          topic:=realsense
-             h_fov:=1.5184351666666667 v_fov:=1.0122901111111111
-             min_range:=0.105          max_range:=8.0
-             width:=640                height:=480
-             update_rate:=30
-             robot_namespace:=/">
-    <!--
-      The gazebo plugin aligns the depth data with the Z axis, with X=left and Y=up
-      ROS expects the depth data along the X axis, with Y=left and Z=up
-      This link only exists to give the gazebo plugin the correctly-oriented frame
-    -->
-    <link name="${frame}_gazebo" />
-    <joint name="${frame}_gazebo_joint" type="fixed">
-      <parent link="${frame}"/>
-      <child link="${frame}_gazebo"/>
-      <origin xyz="0.0 0 0" rpy="-1.5707963267948966 0 -1.5707963267948966"/>
-    </joint>
-    <gazebo reference="${frame}">
-      <turnGravityOff>true</turnGravityOff>
-      <sensor type="depth" name="${prefix}_realsense_depth">
-        <update_rate>${update_rate}</update_rate>
-        <camera>
-          <!-- 75x65 degree FOV for the depth sensor -->
-          <horizontal_fov>${h_fov}</horizontal_fov>
-          <vertical_fov>${v_fov}</vertical_fov>
-          <image>
-            <width>${width}</width>
-            <height>${height}</height>
-            <!-- TODO: check what format the Realsense hardware delivers and set this to match! -->
-            <format>RGB8</format>
-          </image>
-          <clip>
-            <!-- give the color sensor a maximum range of 50m so that the simulation renders nicely -->
-            <near>0.01</near>
-            <far>50.0</far>
-          </clip>
-        </camera>
-        <plugin name="kinect_controller" filename="libgazebo_ros_openni_kinect.so">
-          <baseline>0.2</baseline>
-          <alwaysOn>true</alwaysOn>
-          <updateRate>${update_rate}</updateRate>
-          <cameraName>${topic}</cameraName>
-          <imageTopicName>color/image_raw</imageTopicName>
-          <cameraInfoTopicName>color/camera_info</cameraInfoTopicName>
-          <depthImageTopicName>depth/image_rect_raw</depthImageTopicName>
-          <depthImageInfoTopicName>depth/camera_info</depthImageInfoTopicName>
-          <pointCloudTopicName>depth/color/points</pointCloudTopicName>
-          <frameName>${frame}_gazebo</frameName>
-          <pointCloudCutoff>${min_range}</pointCloudCutoff>
-          <pointCloudCutoffMax>${max_range}</pointCloudCutoffMax>
-          <distortionK1>0.00000001</distortionK1>
-          <distortionK2>0.00000001</distortionK2>
-          <distortionK3>0.00000001</distortionK3>
-          <distortionT1>0.00000001</distortionT1>
-          <distortionT2>0.00000001</distortionT2>
-          <CxPrime>0</CxPrime>
-          <Cx>0</Cx>
-          <Cy>0</Cy>
-          <focalLength>0</focalLength>
-          <hackBaseline>0</hackBaseline>
+  <xacro:macro name="realsense_sensor" params="
+               rs_model:=d435
+               prefix:=front
+               topic:=realsense
+               width:=680
+               height:=480
+               update_rate:=30">
+    <xacro:macro name="realsense_gazebo" params="
+              prefix=front              model=d4
+              frame:=realsense          topic:=realsense
+              h_fov:=1.5184351666666667 v_fov:=1.0122901111111111
+              min_range:=0.105          max_range:=8.0
+              width:=640                height:=480
+              update_rate:=30
+              robot_namespace:=/">
+     <!--
+       The gazebo plugin aligns the depth data with the Z axis, with X=left and Y=up
+       ROS expects the depth data along the X axis, with Y=left and Z=up
+       This link only exists to give the gazebo plugin the correctly-oriented frame
+     -->
+     <link name="${frame}_gazebo" />
+     <joint name="${frame}_gazebo_joint" type="fixed">
+       <parent link="${frame}"/>
+       <child link="${frame}_gazebo"/>
+       <origin xyz="0.0 0 0" rpy="-1.5707963267948966 0 -1.5707963267948966"/>
+     </joint>
+     <gazebo reference="${frame}">
+       <turnGravityOff>true</turnGravityOff>
+       <sensor type="depth" name="${prefix}_realsense_depth">
+         <update_rate>${update_rate}</update_rate>
+         <camera>
+           <!-- 75x65 degree FOV for the depth sensor -->
+           <horizontal_fov>${h_fov}</horizontal_fov>
+           <vertical_fov>${v_fov}</vertical_fov>
+           <image>
+             <width>${width}</width>
+             <height>${height}</height>
+             <!-- TODO: check what format the Realsense hardware delivers and set this to match! -->
+             <format>RGB8</format>
+           </image>
+           <clip>
+             <!-- give the color sensor a maximum range of 50m so that the simulation renders nicely -->
+             <near>0.01</near>
+             <far>50.0</far>
+           </clip>
+         </camera>
+         <plugin name="kinect_controller" filename="libgazebo_ros_openni_kinect.so">
+           <baseline>0.2</baseline>
+           <alwaysOn>true</alwaysOn>
+           <updateRate>${update_rate}</updateRate>
+           <cameraName>${topic}</cameraName>
+           <imageTopicName>color/image_raw</imageTopicName>
+           <cameraInfoTopicName>color/camera_info</cameraInfoTopicName>
+           <depthImageTopicName>depth/image_rect_raw</depthImageTopicName>
+           <depthImageInfoTopicName>depth/camera_info</depthImageInfoTopicName>
+           <pointCloudTopicName>depth/color/points</pointCloudTopicName>
+           <frameName>${frame}_gazebo</frameName>
+           <pointCloudCutoff>${min_range}</pointCloudCutoff>
+           <pointCloudCutoffMax>${max_range}</pointCloudCutoffMax>
+           <distortionK1>0.00000001</distortionK1>
+           <distortionK2>0.00000001</distortionK2>
+           <distortionK3>0.00000001</distortionK3>
+           <distortionT1>0.00000001</distortionT1>
+           <distortionT2>0.00000001</distortionT2>
+           <CxPrime>0</CxPrime>
+           <Cx>0</Cx>
+           <Cy>0</Cy>
+           <focalLength>0</focalLength>
+           <hackBaseline>0</hackBaseline>
+         </plugin>
+       </sensor>
+     </gazebo>
+    </xacro:macro>
+    <xacro:if value="${rs_model == 'd435'}">
+      <xacro:include filename="$(find realsense2_description)/urdf/_d435.urdf.xacro" />
+      <xacro:sensor_d435 parent="${prefix}_mount"
+                        name="${prefix}_realsense">
+        <origin xyz="$(optenv DINGO_REALSENSE_OFFSET 0 0 0)" rpy="$(optenv DINGO_REALSENSE_RPY 0 0 0)" />
+      </xacro:sensor_d435>
+      <xacro:realsense_gazebo
+         prefix="${prefix}"
+         frame="${prefix}_realsense_link"
+         topic="${topic}"
+         h_fov="1.5184351666666667"
+         v_fov="1.0122901111111111"
+         min_range="0.105"
+         max_range="8.0"
+         width="${width}"
+         height="${height}"
+         update_rate="${update_rate}" />
+    </xacro:if>
+    <xacro:if value="${rs_model == 'd435i'}">
+      <xacro:include filename="$(find realsense2_description)/urdf/_d435i.urdf.xacro" />
+      <xacro:sensor_d435i parent="$(optenv DINGO_REALSENSE_MOUNT front)_mount"
+                          name="$(optenv DINGO_REALSENSE_MOUNT front)_realsense">
+        <origin xyz="$(optenv DINGO_REALSENSE_OFFSET 0 0 0)" rpy="$(optenv DINGO_REALSENSE_RPY 0 0 0)" />
+      </xacro:sensor_d435i>
+      <xacro:realsense_gazebo
+         prefix="$(optenv DINGO_REALSENSE_MOUNT front)"
+         frame="$(optenv DINGO_REALSENSE_MOUNT front)_realsense_link"
+         topic="$(optenv DINGO_REALSENSE_TOPIC realsense)"
+         h_fov="1.5184351666666667"
+         v_fov="1.0122901111111111"
+         min_range="0.105"
+         max_range="8.0"
+         width="${width}"
+         height="${height}"
+         update_rate="${update_rate}" />
+      <!--
+        Add the IMU plugin
+        The realsense2_camera driver splits the accelerometer and gyroscope data
+        across 2 topics: accel and gyro
+      -->
+      <gazebo>
+        <plugin name="d435_accel" filename="libhector_gazebo_ros_imu.so">
+          <robotNamespace>/</robotNamespace>
+          <updateRate>30.0</updateRate>
+          <bodyName>$(optenv DINGO_REALSENSE_MOUNT front)_realsense_link</bodyName>
+          <topicName>$(optenv DINGO_REALSENSE_TOPIC realsense)/accel/sample</topicName>
+          <accelDrift>0.005 0.005 0.005</accelDrift>
+          <accelGaussianNoise>0.005 0.005 0.005</accelGaussianNoise>
+          <rateDrift>0.005 0.005 0.005 </rateDrift>
+          <rateGaussianNoise>0.005 0.005 0.005 </rateGaussianNoise>
+          <headingDrift>0.005</headingDrift>
+          <headingGaussianNoise>0.005</headingGaussianNoise>
         </plugin>
-      </sensor>
-    </gazebo>
+        <plugin name="d435_gyro" filename="libhector_gazebo_ros_imu.so">
+          <robotNamespace>/</robotNamespace>
+          <updateRate>30.0</updateRate>
+          <bodyName>$(optenv DINGO_REALSENSE_MOUNT front)_realsense_link</bodyName>
+          <topicName>$(optenv DINGO_REALSENSE_TOPIC realsense)/gyro/sample</topicName>
+          <accelDrift>0.005 0.005 0.005</accelDrift>
+          <accelGaussianNoise>0.005 0.005 0.005</accelGaussianNoise>
+          <rateDrift>0.005 0.005 0.005 </rateDrift>
+          <rateGaussianNoise>0.005 0.005 0.005 </rateGaussianNoise>
+          <headingDrift>0.005</headingDrift>
+          <headingGaussianNoise>0.005</headingGaussianNoise>
+        </plugin>
+      </gazebo>
+    </xacro:if>
+    <xacro:if value="${rs_model == 'd415'}">
+      <xacro:include filename="$(find realsense2_description)/urdf/_d415.urdf.xacro" />
+      <xacro:sensor_d415 parent="$(optenv DINGO_REALSENSE_MOUNT front)_mount"
+                         name="$(optenv DINGO_REALSENSE_MOUNT front)_realsense">
+        <origin xyz="$(optenv DINGO_REALSENSE_OFFSET 0 0 0)" rpy="$(optenv DINGO_REALSENSE_RPY 0 0 0)" />
+      </xacro:sensor_d415>
+      <xacro:realsense_gazebo
+         prefix="$(optenv DINGO_REALSENSE_MOUNT front)"
+         frame="$(optenv DINGO_REALSENSE_MOUNT front)_realsense_link"
+         topic="$(optenv DINGO_REALSENSE_TOPIC realsense)"
+         h_fov="1.1344640137963142"
+         v_fov="0.6981317007977318"
+         min_range="0.3"
+         max_range="5.0"
+         width="${width}"
+         height="${height}"
+         update_rate="${update_rate}" />
+    </xacro:if>
+    <xacro:if value="${rs_model == 'd455'}">
+      <!-- TODO: not officially supported yet. Use the D435 mesh for now, even though it's the wrong size -->
+      <xacro:include filename="$(find realsense2_description)/urdf/_d435.urdf.xacro" />
+      <xacro:sensor_d435 parent="$(optenv DINGO_REALSENSE_MOUNT front)_mount"
+                         name="$(optenv DINGO_REALSENSE_MOUNT front)_realsense">
+        <origin xyz="$(optenv DINGO_REALSENSE_OFFSET 0 0 0)" rpy="$(optenv DINGO_REALSENSE_RPY 0 0 0)" />
+      </xacro:sensor_d435>
+      <xacro:realsense_gazebo
+         prefix="$(optenv DINGO_REALSENSE_MOUNT front)"
+         frame="$(optenv DINGO_REALSENSE_MOUNT front)_realsense_link"
+         topic="$(optenv DINGO_REALSENSE_TOPIC realsense)"
+         h_fov="1.5009831567151233"
+         v_fov="0.9948376736367678"
+         min_range="0.5"
+         max_range="20.0"
+         width="${width}"
+         height="${height}"
+         update_rate="${update_rate}" />
+    </xacro:if>
+    <xacro:if value="${rs_model == 'l515'}">
+      <!--
+        TODO: not officially supported yet.
+        Because the camera is a radically different shape, rather than use the D435 or D415 mesh, create
+        the shape of the sensor manually.  This will be a rough approximation only
+      -->
+      <link name="${prefix}_realsense_bottom_screw_frame">
+        <visual>
+          <origin xyz="0 0 0.0305" rpy="0 ${PI/2} 0"/>
+          <geometry>
+            <cylinder radius="0.0305" length="0.026" />
+          </geometry>
+          <material name="white">
+            <color rgba="1 1 1 1" />
+          </material>
+        </visual>
+      </link>
+      <link name="${prefix}_realsense_link">
+        <visual>
+          <origin xyz="0.001 0 0" rpy="0 ${PI/2} 0"/>
+          <geometry>
+            <cylinder radius="0.0295" length="0.026"/>
+          </geometry>
+          <material name="black" />
+        </visual>
+      </link>
+      <joint type="fixed" name="${prefix}_realsense_ring_to_lens">
+        <parent link="${prefix}_realsense_bottom_screw_frame" />
+        <child link="${prefix}_realsense_link" />
+        <origin xyz="0 0 0.0305" rpy="0 0 0" />
+      </joint>
+      <joint type="fixed" name="${prefix}_realsense_mount_joint">
+        <parent link="${prefix}_mount" />
+        <child link="${prefix}_realsense_bottom_screw_frame" />
+        <origin xyz="0 0 0.004" rpy="0 0 0" />
+      </joint>
+      <xacro:realsense_gazebo
+         prefix="$(optenv DINGO_REALSENSE_MOUNT front)"
+         frame="$(optenv DINGO_REALSENSE_MOUNT front)_realsense_link"
+         topic="$(optenv DINGO_REALSENSE_TOPIC realsense)"
+         h_fov="1.2217304763960306"
+         v_fov="0.9599310885968813"
+         min_range="0.25"
+         max_range="9.0"
+         width="${width}"
+         height="${height}"
+         update_rate="${update_rate}" />
+    </xacro:if>
   </xacro:macro>
 </robot>
