Commit message: Nav improvements (#5)
* Expose the scan_topic argument in the gmapping_demo and amcl_demo launch files

* Add placeholder support for the RS L515 and D455 so that the gazebo plugins work; the meshes for these sensors don't exist yet, but we can at least get the plugin configured & add the appropriate links for now

* Refactor the RealSense macro to put the mesh + gazebo plugin in one place. Create a more-accurate L515 mesh out of cylinders until Intel releases an official mesh for the sensor

File: dingo_description/urdf/accessories.urdf.xacro (robot description, xacro)
@@ -50,99 +50,8 @@
   -->
   <xacro:if value="$(optenv DINGO_REALSENSE 0)">
-    <xacro:property name="rs_model" value="$(optenv DINGO_REALSENSE_MODEL d435)" />
-    <xacro:if value="${rs_model == 'd435'}">
-      <xacro:include filename="$(find realsense2_description)/urdf/_d435.urdf.xacro" />
-      <xacro:sensor_d435 parent="$(optenv DINGO_REALSENSE_MOUNT front)_mount"
-                         name="$(optenv DINGO_REALSENSE_MOUNT front)_realsense">
-        <origin xyz="$(optenv DINGO_REALSENSE_OFFSET 0 0 0)" rpy="$(optenv DINGO_REALSENSE_RPY 0 0 0)" />
-      </xacro:sensor_d435>
-      <include filename="$(find dingo_description)/urdf/accessories/intel_realsense.urdf.xacro" />
-      <xacro:realsense_gazebo
-        prefix="$(optenv DINGO_REALSENSE_MOUNT front)"
-        frame="$(optenv DINGO_REALSENSE_MOUNT front)_realsense_link"
-        topic="$(optenv DINGO_REALSENSE_TOPIC realsense)"
-        h_fov="1.5184351666666667"
-        v_fov="1.0122901111111111"
-        min_range="0.105"
-        max_range="8.0"
-        width="640"
-        height="480"
-        update_rate="30" />
-    </xacro:if>
-    <xacro:if value="${rs_model == 'd435i'}">
-      <xacro:include filename="$(find realsense2_description)/urdf/_d435i.urdf.xacro" />
-      <xacro:sensor_d435i parent="$(optenv DINGO_REALSENSE_MOUNT front)_mount"
-                         name="$(optenv DINGO_REALSENSE_MOUNT front)_realsense">
-        <origin xyz="$(optenv DINGO_REALSENSE_OFFSET 0 0 0)" rpy="$(optenv DINGO_REALSENSE_RPY 0 0 0)" />
-      </xacro:sensor_d435i>
-      <include filename="$(find dingo_description)/urdf/accessories/intel_realsense.urdf.xacro" />
-      <xacro:realsense_gazebo
-        prefix="$(optenv DINGO_REALSENSE_MOUNT front)"
-        frame="$(optenv DINGO_REALSENSE_MOUNT front)_realsense_link"
-        topic="$(optenv DINGO_REALSENSE_TOPIC realsense)"
-        h_fov="1.5184351666666667"
-        v_fov="1.0122901111111111"
-        min_range="0.105"
-        max_range="8.0"
-        width="640"
-        height="480"
-        update_rate="30" />
-      <!--
-        Add the IMU plugin
-        The realsense2_camera driver splits the accelerometer and gyroscope data
-        across 2 topics: accel and gyro
-      -->
-      <gazebo>
-        <plugin name="d435_accel" filename="libhector_gazebo_ros_imu.so">
-          <robotNamespace>/</robotNamespace>
-          <updateRate>30.0</updateRate>
-          <bodyName>$(optenv DINGO_REALSENSE_MOUNT front)_realsense_link</bodyName>
-          <topicName>$(optenv DINGO_REALSENSE_TOPIC realsense)/accel/sample</topicName>
-          <accelDrift>0.005 0.005 0.005</accelDrift>
-          <accelGaussianNoise>0.005 0.005 0.005</accelGaussianNoise>
-          <rateDrift>0.005 0.005 0.005 </rateDrift>
-          <rateGaussianNoise>0.005 0.005 0.005 </rateGaussianNoise>
-          <headingDrift>0.005</headingDrift>
-          <headingGaussianNoise>0.005</headingGaussianNoise>
-        </plugin>
-        <plugin name="d435_gyro" filename="libhector_gazebo_ros_imu.so">
-          <robotNamespace>/</robotNamespace>
-          <updateRate>30.0</updateRate>
-          <bodyName>$(optenv DINGO_REALSENSE_MOUNT front)_realsense_link</bodyName>
-          <topicName>$(optenv DINGO_REALSENSE_TOPIC realsense)/gyro/sample</topicName>
-          <accelDrift>0.005 0.005 0.005</accelDrift>
-          <accelGaussianNoise>0.005 0.005 0.005</accelGaussianNoise>
-          <rateDrift>0.005 0.005 0.005 </rateDrift>
-          <rateGaussianNoise>0.005 0.005 0.005 </rateGaussianNoise>
-          <headingDrift>0.005</headingDrift>
-          <headingGaussianNoise>0.005</headingGaussianNoise>
-        </plugin>
-      </gazebo>
-    </xacro:if>
-    <xacro:if value="${rs_model == 'd415'}">
-      <xacro:include filename="$(find realsense2_description)/urdf/_d415.urdf.xacro" />
-      <xacro:sensor_d415 parent="$(optenv DINGO_REALSENSE_MOUNT front)_mount"
-                         name="$(optenv DINGO_REALSENSE_MOUNT front)_realsense">
-        <origin xyz="$(optenv DINGO_REALSENSE_OFFSET 0 0 0)" rpy="$(optenv DINGO_REALSENSE_RPY 0 0 0)" />
-      </xacro:sensor_d415>
-      <include filename="$(find dingo_description)/urdf/accessories/intel_realsense.urdf.xacro" />
-      <xacro:realsense_gazebo
-        prefix="$(optenv DINGO_REALSENSE_MOUNT front)"
-        frame="$(optenv DINGO_REALSENSE_MOUNT front)_realsense_link"
-        topic="$(optenv DINGO_REALSENSE_TOPIC realsense)"
-        h_fov="1.1344640137963142"
-        v_fov="0.6981317007977318"
-        min_range="0.3"
-        max_range="5.0"
-        width="640"
-        height="480"
-        update_rate="30" />
-    </xacro:if>
-    <xacro:if value="${rs_model == 'd455'}">
-      <!-- TODO: not officially supported yet -->
-    </xacro:if>
-    <xacro:if value="${rs_model == 'l515'}">
-      <!-- TODO: not officially supported yet -->
-    </xacro:if>
+    <include filename="$(find dingo_description)/urdf/accessories/intel_realsense.urdf.xacro" />
+    <xacro:realsense_sensor rs_model="$(optenv DINGO_REALSENSE_MODEL d435)"
+                            prefix="$(optenv DINGO_REALSENSE_MOUNT front)"
+                            topic="$(optenv DINGO_REALSENSE_TOPIC realsense)" />
   </xacro:if>
 </robot>

Commit message: Add support for the VLP16 as a standard laser sensor on this platform

File: dingo_description/urdf/accessories.urdf.xacro (robot description, xacro)
@@ -39,4 +39,10 @@
       </joint>
     </xacro:if>
+    <xacro:if value="${lidar_model == 'vlp16'}">
+      <xacro:include filename="$(find velodyne_description)/urdf/VLP-16.urdf.xacro" />
+      <xacro:VLP-16 parent="$(optenv DINGO_LASER_MOUNT front)_mount" topic="$(optenv DINGO_LASER_TOPIC front/points)">
+        <origin xyz="$(optenv DINGO_LASER_OFFSET 0 0 0)" rpy="$(optenv DINGO_LASER_RPY 0 0 0)" />
+      </xacro:VLP-16>
+    </xacro:if>
   </xacro:if>
   <!--

Commit message: Add the 3D and secondary 2D lidars

File: dingo_description/urdf/accessories.urdf.xacro (robot description, xacro)
@@ -9,4 +9,7 @@
     dingo_base/launch/base.launch
   -->
+  <xacro:include filename="$(find dingo_description)/urdf/accessories/sick_lms1xx_mount.urdf.xacro" />
+  <xacro:include filename="$(find dingo_description)/urdf/accessories/hokuyo_ust10.urdf.xacro" />
+  <xacro:include filename="$(find dingo_description)/urdf/accessories/vlp16_mount.urdf.xacro" />
   <!--
     Add a lidar sensor.  By default this is a SICK LMS1xx but can be changed with the
@@ -14,10 +17,8 @@
     - lms1xx (default) :: SICK LMS1xx
     - ust10            :: Hokuyo UST10
-    - vlp16            :: Velodyne VLP16
   -->
   <xacro:if value="$(optenv DINGO_LASER 0)">
     <xacro:property name="lidar_model" value="$(optenv DINGO_LASER_MODEL lms1xx)" />
     <xacro:if value="${lidar_model == 'lms1xx'}">
-      <xacro:include filename="$(find dingo_description)/urdf/accessories/sick_lms1xx_mount.urdf.xacro" />
       <xacro:sick_lms1xx_mount prefix="$(optenv DINGO_LASER_MOUNT front)"
                          topic="$(optenv DINGO_LASER_TOPIC front/scan)"/>
@@ -30,5 +31,4 @@
     </xacro:if>
     <xacro:if value="${lidar_model == 'ust10'}">
-      <xacro:include filename="$(find dingo_description)/urdf/accessories/hokuyo_ust10.urdf.xacro" />
       <xacro:hokuyo_ust10_mount prefix="$(optenv DINGO_LASER_MOUNT front)"
                           topic="$(optenv DINGO_LASER_TOPIC front/scan)" />
@@ -40,9 +40,43 @@
       </joint>
     </xacro:if>
-    <xacro:if value="${lidar_model == 'vlp16'}">
-      <xacro:include filename="$(find velodyne_description)/urdf/VLP-16.urdf.xacro" />
-      <xacro:VLP-16 parent="$(optenv DINGO_LASER_MOUNT front)_mount" topic="$(optenv DINGO_LASER_TOPIC front/points)">
-        <origin xyz="$(optenv DINGO_LASER_OFFSET 0 0 0)" rpy="$(optenv DINGO_LASER_RPY 0 0 0)" />
-      </xacro:VLP-16>
+  </xacro:if>
+  <!-- Add the secondary lidar, same format as the first, but on the rear -->
+  <xacro:if value="$(optenv DINGO_LASER_SECONDARY 0)">
+    <xacro:property name="lidar2_model" value="$(optenv DINGO_LASER_SECONDARY_MODEL lms1xx)" />
+    <xacro:if value="${lidar2_model == 'lms1xx'}">
+      <xacro:sick_lms1xx_mount prefix="$(optenv DINGO_LASER_SECONDARY_MOUNT rear)"
+                         topic="$(optenv DINGO_LASER_SECONDARY_TOPIC rear/scan)"/>
+      <joint name="$(optenv DINGO_LASER_SECONDARY_MOUNT rear)_laser_mount_joint" type="fixed">
+        <origin xyz="$(optenv DINGO_LASER_SECONDARY_OFFSET 0 0 0)"
+                rpy="$(optenv DINGO_LASER_SECONDARY_RPY 0 0 ${M_PI})" />
+        <parent link="$(optenv DINGO_LASER_SECONDARY_MOUNT rear)_mount" />
+        <child link="$(optenv DINGO_LASER_SECONDARY_MOUNT rear)_laser_mount" />
+      </joint>
+    </xacro:if>
+    <xacro:if value="${lidar2_model == 'ust10'}">
+      <xacro:hokuyo_ust10_mount prefix="$(optenv DINGO_LASER_SECONDARY_MOUNT rear)"
+                          topic="$(optenv DINGO_LASER_SECONDARY_TOPIC rear/scan)" />
+      <joint name="$(optenv DINGO_LASER_SECONDARY_MOUNT rear)_laser_mount_joint" type="fixed">
+        <origin xyz="$(optenv DINGO_LASER_SECONDARY_OFFSET 0 0 0)"
+                rpy="$(optenv DINGO_LASER_SECONDARY_RPY 0 0 ${M_PI})" />
+        <parent link="$(optenv DINGO_LASER_SECONDARY_MOUNT rear)_mount" />
+        <child link="$(optenv DINGO_LASER_SECONDARY_MOUNT rear)_laser_mount" />
+      </joint>
+    </xacro:if>
+  </xacro:if>
+  <!--
+    Add a 3D lidar sensor.  By default this is a VLP16 but can be changed with the
+    DINGO_LASER_3D_MODEL environment variable. Valid model designations are:
+    - vlp16 (default) :: Velodyne VLP16=
+  -->
+  <xacro:if value="$(optenv DINGO_LASER_3D 0)">
+    <xacro:property name="lidar_3d_model" value="$(optenv DINGO_LASER_3D_MODEL vlp16)" />
+    <xacro:if value="${lidar_3d_model == 'vlp16'}">
+      <xacro:vlp16_mount
+          prefix="$(optenv DINGO_LASER_3D_MOUNT front)"
+          parent_link="$(optenv DINGO_LASER_3D_MOUNT front)_mount"
+          topic="$(optenv DINGO_LASER_3D_TOPIC front/points)">
+        <origin xyz="$(optenv DINGO_LASER_3D_OFFSET 0 0 0)" rpy="$(optenv DINGO_LASER_3D_RPY 0 0 0)" />
+      </xacro:vlp16_mount>
     </xacro:if>
   </xacro:if>

Commit message: Add env var support for VLP-16 (#10)
* Add support for the VLP16 as a standard laser sensor on this platform

* Add vlp16 to the comment block explaining supported laser scanners

* Add the 3D and secondary 2D lidars

File: dingo_description/urdf/accessories.urdf.xacro (robot description, xacro)
@@ -9,4 +9,7 @@
     dingo_base/launch/base.launch
   -->
+  <xacro:include filename="$(find dingo_description)/urdf/accessories/sick_lms1xx_mount.urdf.xacro" />
+  <xacro:include filename="$(find dingo_description)/urdf/accessories/hokuyo_ust10.urdf.xacro" />
+  <xacro:include filename="$(find dingo_description)/urdf/accessories/vlp16_mount.urdf.xacro" />
   <!--
     Add a lidar sensor.  By default this is a SICK LMS1xx but can be changed with the
@@ -18,5 +21,4 @@
     <xacro:property name="lidar_model" value="$(optenv DINGO_LASER_MODEL lms1xx)" />
     <xacro:if value="${lidar_model == 'lms1xx'}">
-      <xacro:include filename="$(find dingo_description)/urdf/accessories/sick_lms1xx_mount.urdf.xacro" />
       <xacro:sick_lms1xx_mount prefix="$(optenv DINGO_LASER_MOUNT front)"
                          topic="$(optenv DINGO_LASER_TOPIC front/scan)"/>
@@ -29,5 +31,4 @@
     </xacro:if>
     <xacro:if value="${lidar_model == 'ust10'}">
-      <xacro:include filename="$(find dingo_description)/urdf/accessories/hokuyo_ust10.urdf.xacro" />
       <xacro:hokuyo_ust10_mount prefix="$(optenv DINGO_LASER_MOUNT front)"
                           topic="$(optenv DINGO_LASER_TOPIC front/scan)" />
@@ -38,4 +39,44 @@
         <child link="$(optenv DINGO_LASER_MOUNT front)_laser_mount" />
       </joint>
+    </xacro:if>
+  </xacro:if>
+  <!-- Add the secondary lidar, same format as the first, but on the rear -->
+  <xacro:if value="$(optenv DINGO_LASER_SECONDARY 0)">
+    <xacro:property name="lidar2_model" value="$(optenv DINGO_LASER_SECONDARY_MODEL lms1xx)" />
+    <xacro:if value="${lidar2_model == 'lms1xx'}">
+      <xacro:sick_lms1xx_mount prefix="$(optenv DINGO_LASER_SECONDARY_MOUNT rear)"
+                         topic="$(optenv DINGO_LASER_SECONDARY_TOPIC rear/scan)"/>
+      <joint name="$(optenv DINGO_LASER_SECONDARY_MOUNT rear)_laser_mount_joint" type="fixed">
+        <origin xyz="$(optenv DINGO_LASER_SECONDARY_OFFSET 0 0 0)"
+                rpy="$(optenv DINGO_LASER_SECONDARY_RPY 0 0 ${M_PI})" />
+        <parent link="$(optenv DINGO_LASER_SECONDARY_MOUNT rear)_mount" />
+        <child link="$(optenv DINGO_LASER_SECONDARY_MOUNT rear)_laser_mount" />
+      </joint>
+    </xacro:if>
+    <xacro:if value="${lidar2_model == 'ust10'}">
+      <xacro:hokuyo_ust10_mount prefix="$(optenv DINGO_LASER_SECONDARY_MOUNT rear)"
+                          topic="$(optenv DINGO_LASER_SECONDARY_TOPIC rear/scan)" />
+      <joint name="$(optenv DINGO_LASER_SECONDARY_MOUNT rear)_laser_mount_joint" type="fixed">
+        <origin xyz="$(optenv DINGO_LASER_SECONDARY_OFFSET 0 0 0)"
+                rpy="$(optenv DINGO_LASER_SECONDARY_RPY 0 0 ${M_PI})" />
+        <parent link="$(optenv DINGO_LASER_SECONDARY_MOUNT rear)_mount" />
+        <child link="$(optenv DINGO_LASER_SECONDARY_MOUNT rear)_laser_mount" />
+      </joint>
+    </xacro:if>
+  </xacro:if>
+  <!--
+    Add a 3D lidar sensor.  By default this is a VLP16 but can be changed with the
+    DINGO_LASER_3D_MODEL environment variable. Valid model designations are:
+    - vlp16 (default) :: Velodyne VLP16=
+  -->
+  <xacro:if value="$(optenv DINGO_LASER_3D 0)">
+    <xacro:property name="lidar_3d_model" value="$(optenv DINGO_LASER_3D_MODEL vlp16)" />
+    <xacro:if value="${lidar_3d_model == 'vlp16'}">
+      <xacro:vlp16_mount
+          prefix="$(optenv DINGO_LASER_3D_MOUNT front)"
+          parent_link="$(optenv DINGO_LASER_3D_MOUNT front)_mount"
+          topic="$(optenv DINGO_LASER_3D_TOPIC front/points)">
+        <origin xyz="$(optenv DINGO_LASER_3D_OFFSET 0 0 0)" rpy="$(optenv DINGO_LASER_3D_RPY 0 0 0)" />
+      </xacro:vlp16_mount>
     </xacro:if>
   </xacro:if>
