Commit message: Updated URDF to disable mount

File: dingo_description/urdf/accessories.urdf.xacro (robot description, xacro)
@@ -11,4 +11,5 @@
   <xacro:include filename="$(find dingo_description)/urdf/accessories/sick_lms1xx_mount.urdf.xacro" />
   <xacro:include filename="$(find dingo_description)/urdf/accessories/hokuyo_ust10.urdf.xacro" />
+  <xacro:include filename="$(find dingo_description)/urdf/accessories/hdl32_mount.urdf.xacro" />
   <xacro:include filename="$(find dingo_description)/urdf/accessories/vlp16_mount.urdf.xacro" />
   <!--
@@ -19,23 +20,47 @@
   -->
   <xacro:if value="$(optenv DINGO_LASER 0)">
+    <xacro:property name="mount" value="$(optenv DINGO_LASER_MOUNT front)" />
+    <xacro:property name="topic" value="$(optenv DINGO_LASER_TOPIC front/scan)" />
+    <xacro:property name="tower" value="$(optenv DINGO_LASER_TOWER 1)" />
+    <xacro:property name="prefix" value="$(optenv DINGO_LASER_PREFIX ${mount})" />
+    <xacro:property name="parent" value="$(optenv DINGO_LASER_PARENT ${mount}_mount)" />
     <xacro:property name="lidar_model" value="$(optenv DINGO_LASER_MODEL lms1xx)" />
+    <!-- SICK LMS1xx -->
     <xacro:if value="${lidar_model == 'lms1xx'}">
-      <xacro:sick_lms1xx_mount prefix="$(optenv DINGO_LASER_MOUNT front)"
-                         topic="$(optenv DINGO_LASER_TOPIC front/scan)"/>
-      <joint name="$(optenv DINGO_LASER_MOUNT front)_laser_mount_joint" type="fixed">
+      <!-- Mount Enabled -->
+      <xacro:if value="${tower}">
+        <xacro:sick_lms1xx_mount prefix="${prefix}" topic="${topic}"/>
+        <joint name="${prefix}_laser_mount_joint" type="fixed">
+          <origin xyz="$(optenv DINGO_LASER_OFFSET 0 0 0)"
+                  rpy="$(optenv DINGO_LASER_RPY 0 0 0)" />
+          <parent link="${parent}" />
+          <child link="${prefix}_laser_mount" />
+        </joint>
+      </xacro:if>
+      <!-- Mount Disabled -->
+      <xacro:unless value="${tower}">
+        <xacro:sick_lms1xx frame="${prefix}_laser" topic="${topic}" />
+        <link name="${prefix}_laser_base"/>
+        <joint name="${prefix}_laser_base_joint" type="fixed">
+          <origin xyz="$(optenv DINGO_LASER_OFFSET 0 0 0)"
+                  rpy="$(optenv DINGO_LASER_RPY 0 0 0)"/>
+          <parent link="${parent}"/>
+          <child link="${prefix}_laser_base"/>
+        </joint>
+        <joint name="${prefix}_laser_joint" type="fixed">
+          <origin xyz="0 0 0.116" rpy="0 0 0"/>
+          <parent link="${prefix}_laser_base"/>
+          <child link="${prefix}_laser"/>
+        </joint>
+      </xacro:unless>
+    </xacro:if>
+    <!-- Hokuyo UST10 -->
+    <xacro:if value="${lidar_model == 'ust10'}">
+      <xacro:hokuyo_ust10_mount prefix="${prefix}" topic="${topic}" />
+      <joint name="${prefix}_laser_mount_joint" type="fixed">
         <origin xyz="$(optenv DINGO_LASER_OFFSET 0 0 0)"
                 rpy="$(optenv DINGO_LASER_RPY 0 0 0)" />
-        <parent link="$(optenv DINGO_LASER_MOUNT front)_mount" />
-        <child link="$(optenv DINGO_LASER_MOUNT front)_laser_mount" />
-      </joint>
-    </xacro:if>
-    <xacro:if value="${lidar_model == 'ust10'}">
-      <xacro:hokuyo_ust10_mount prefix="$(optenv DINGO_LASER_MOUNT front)"
-                          topic="$(optenv DINGO_LASER_TOPIC front/scan)" />
-      <joint name="$(optenv DINGO_LASER_MOUNT front)_laser_mount_joint" type="fixed">
-        <origin xyz="$(optenv DINGO_LASER_OFFSET 0 0 0)"
-                rpy="$(optenv DINGO_LASER_RPY 0 0 0)" />
-        <parent link="$(optenv DINGO_LASER_MOUNT front)_mount" />
-        <child link="$(optenv DINGO_LASER_MOUNT front)_laser_mount" />
+        <parent link="${parent}" />
+        <child link="${prefix}_laser_mount" />
       </joint>
     </xacro:if>
@@ -43,23 +68,47 @@
   <!-- Add the secondary lidar, same format as the first, but on the rear -->
   <xacro:if value="$(optenv DINGO_LASER_SECONDARY 0)">
-    <xacro:property name="lidar2_model" value="$(optenv DINGO_LASER_SECONDARY_MODEL lms1xx)" />
-    <xacro:if value="${lidar2_model == 'lms1xx'}">
-      <xacro:sick_lms1xx_mount prefix="$(optenv DINGO_LASER_SECONDARY_MOUNT rear)"
-                         topic="$(optenv DINGO_LASER_SECONDARY_TOPIC rear/scan)"/>
-      <joint name="$(optenv DINGO_LASER_SECONDARY_MOUNT rear)_laser_mount_joint" type="fixed">
+    <xacro:property name="mount" value="$(optenv DINGO_LASER_SECONDARY_MOUNT rear)" />
+    <xacro:property name="topic" value="$(optenv DINGO_LASER_SECONDARY_TOPIC rear/scan)" />
+    <xacro:property name="tower" value="$(optenv DINGO_LASER_SECONDARY_TOWER 1)" />
+    <xacro:property name="prefix" value="$(optenv DINGO_LASER_SECONDARY_PREFIX ${mount})" />
+    <xacro:property name="parent" value="$(optenv DINGO_LASER_SECONDARY_PARENT ${mount}_mount)" />
+    <xacro:property name="lidar_model" value="$(optenv DINGO_LASER_SECONDARY_MODEL lms1xx)" />
+    <!-- Secondary SICK LMS1xx -->
+    <xacro:if value="${lidar_model == 'lms1xx'}">
+      <!-- Mount Enabled -->
+      <xacro:if value="${tower}">
+        <xacro:sick_lms1xx_mount prefix="${prefix}" topic="${topic}"/>
+        <joint name="${prefix}_laser_mount_joint" type="fixed">
+          <origin xyz="$(optenv DINGO_LASER_SECONDARY_OFFSET 0 0 0)"
+                  rpy="$(optenv DINGO_LASER_SECONDARY_RPY 0 0 ${M_PI})" />
+          <parent link="${parent}" />
+          <child link="${prefix}_laser_mount" />
+        </joint>
+      </xacro:if>
+      <!-- Mount Disabled -->
+      <xacro:unless value="${tower}">
+        <xacro:sick_lms1xx frame="${prefix}_laser" topic="${topic}" />
+        <link name="${prefix}_laser_base"/>
+        <joint name="${prefix}_laser_base_joint" type="fixed">
+          <origin xyz="$(optenv DINGO_LASER_SECONDARY_OFFSET 0 0 0)"
+                  rpy="$(optenv DINGO_LASER_SECONDARY_RPY 0 0 ${M_PI})" />
+          <parent link="${parent}"/>
+          <child link="${prefix}_laser_base"/>
+        </joint>
+        <joint name="${prefix}_laser_joint" type="fixed">
+          <origin xyz="0 0 0.116" rpy="0 0 0"/>
+          <parent link="${prefix}_laser_base"/>
+          <child link="${prefix}_laser"/>
+        </joint>
+      </xacro:unless>
+    </xacro:if>
+    <!-- Secondary Hokuyo UST10 -->
+    <xacro:if value="${lidar_model == 'ust10'}">
+      <xacro:hokuyo_ust10_mount prefix="${prefix}" topic="${topic}" />
+      <joint name="${prefix}_laser_mount_joint" type="fixed">
         <origin xyz="$(optenv DINGO_LASER_SECONDARY_OFFSET 0 0 0)"
                 rpy="$(optenv DINGO_LASER_SECONDARY_RPY 0 0 ${M_PI})" />
-        <parent link="$(optenv DINGO_LASER_SECONDARY_MOUNT rear)_mount" />
-        <child link="$(optenv DINGO_LASER_SECONDARY_MOUNT rear)_laser_mount" />
-      </joint>
-    </xacro:if>
-    <xacro:if value="${lidar2_model == 'ust10'}">
-      <xacro:hokuyo_ust10_mount prefix="$(optenv DINGO_LASER_SECONDARY_MOUNT rear)"
-                          topic="$(optenv DINGO_LASER_SECONDARY_TOPIC rear/scan)" />
-      <joint name="$(optenv DINGO_LASER_SECONDARY_MOUNT rear)_laser_mount_joint" type="fixed">
-        <origin xyz="$(optenv DINGO_LASER_SECONDARY_OFFSET 0 0 0)"
-                rpy="$(optenv DINGO_LASER_SECONDARY_RPY 0 0 ${M_PI})" />
-        <parent link="$(optenv DINGO_LASER_SECONDARY_MOUNT rear)_mount" />
-        <child link="$(optenv DINGO_LASER_SECONDARY_MOUNT rear)_laser_mount" />
+        <parent link="${parent}" />
+        <child link="${prefix}_laser_mount" />
       </joint>
     </xacro:if>
@@ -71,12 +120,22 @@
   -->
   <xacro:if value="$(optenv DINGO_LASER_3D 0)">
+    <xacro:property name="mount" value="$(optenv DINGO_LASER_3D_MOUNT front)" />
+    <xacro:property name="topic" value="$(optenv DINGO_LASER_3D_TOPIC front/points)" />
+    <xacro:property name="tower" value="$(optenv DINGO_LASER_3D_TOWER 1)" />
+    <xacro:property name="angle" value="$(optenv DINGO_LASER_3D_ANGLE 0)" />
+    <xacro:property name="prefix" value="$(optenv DINGO_LASER_3D_PREFIX ${mount})" />
+    <xacro:property name="parent" value="$(optenv DINGO_LASER_3D_PARENT ${mount}_mount)" />
     <xacro:property name="lidar_3d_model" value="$(optenv DINGO_LASER_3D_MODEL vlp16)" />
+    <!-- Velodyne VLP16 -->
     <xacro:if value="${lidar_3d_model == 'vlp16'}">
-      <xacro:vlp16_mount
-          prefix="$(optenv DINGO_LASER_3D_MOUNT front)"
-          parent_link="$(optenv DINGO_LASER_3D_MOUNT front)_mount"
-          topic="$(optenv DINGO_LASER_3D_TOPIC front/points)">
+      <xacro:vlp16_mount topic="${topic}" tower="${tower}" angle="${angle}" prefix="${prefix}" parent_link="${parent}" >
         <origin xyz="$(optenv DINGO_LASER_3D_OFFSET 0 0 0)" rpy="$(optenv DINGO_LASER_3D_RPY 0 0 0)" />
       </xacro:vlp16_mount>
+    </xacro:if>
+    <!-- Velodyne HDL-32E -->
+    <xacro:if value="${lidar_3d_model == 'hdl32e'}">
+      <xacro:hdl32e_mount topic="${topic}" tower="${tower}" angle="${angle}" prefix="${prefix}" parent_link="${parent}" >
+        <origin xyz="$(optenv DINGO_LASER_3D_OFFSET 0 0 0)" rpy="$(optenv DINGO_LASER_3D_RPY 0 0 0)" />
+      </xacro:hdl32e_mount>
     </xacro:if>
   </xacro:if>

Commit message: Added Velodyne HDL32E and Microstrain GX5

File: dingo_description/urdf/accessories.urdf.xacro (robot description, xacro)
@@ -155,3 +155,19 @@
                             topic="$(optenv DINGO_REALSENSE_TOPIC realsense)" />
   </xacro:if>
+  <!--
+    Add Microstrain IMU. By default the DINGO comes equipped with an IMU linked to "imu_link". These extra
+    optional microstrain IMU's will be added to another frame, by default, "microstrain_link".
+  -->
+  <xacro:if value="$(optenv DINGO_IMU_MICROSTRAIN 0)">
+    <xacro:property name="frame"  value="$(optenv DINGO_IMU_MICROSTRAIN_LINK microstrain_link)"/>
+    <xacro:property name="parent" value="$(optenv DINGO_IMU_MICROSTRAIN_PARENT imu_link)"/>
+    <xacro:property name="xyz"    value="$(optenv DINGO_IMU_MICROSTRAIN_OFFSET 0 0 0)"/>
+    <xacro:property name="rpy"    value="$(optenv DINGO_IMU_MICROSTRAIN_RPY 0 0 0)"/>
+    <link name="${frame}" />
+    <joint name="${frame}_joint" type="fixed">
+      <parent link="${parent}" />
+      <child link="${frame}" />
+      <origin xyz="${xyz}" rpy="${rpy}" />
+    </joint>
+  </xacro:if>
 </robot>

Commit message: Added secondary realsense

File: dingo_description/urdf/accessories.urdf.xacro (robot description, xacro)
@@ -148,10 +148,54 @@
     - d455
     - l515
-  -->
-  <xacro:if value="$(optenv DINGO_REALSENSE 0)">
-    <xacro:include filename="$(find dingo_description)/urdf/accessories/intel_realsense.urdf.xacro" />
-    <xacro:realsense_sensor rs_model="$(optenv DINGO_REALSENSE_MODEL d435)"
-                            prefix="$(optenv DINGO_REALSENSE_MOUNT front)"
-                            topic="$(optenv DINGO_REALSENSE_TOPIC realsense)" />
+    Note: If two realsense's are included, both must be the same model type.
+  -->
+  <xacro:include filename="$(find dingo_description)/urdf/accessories/intel_realsense.urdf.xacro" />
+  <xacro:property name="realsense_enabled" value="$(optenv DINGO_REALSENSE 0)"/>
+  <!-- Primary Realsense Parameters -->
+  <xacro:property name="rs_model"   default="$(optenv DINGO_REALSENSE_MODEL d435)"/>
+  <xacro:property name="rs_topic"   default="$(optenv DINGO_REALSENSE_TOPIC realsense)" />
+  <xacro:property name="rs_mount"   default="$(optenv DINGO_REALSENSE_MOUNT front)" />
+  <xacro:property name="rs_prefix"  default="$(optenv DINGO_REALSENSE_PREFIX ${rs_mount})" />
+  <xacro:property name="rs_parent"  default="$(optenv DINGO_REALSENSE_PARENT ${rs_mount}_mount)" />
+  <xacro:property name="rs_xyz"     default="$(optenv DINGO_REALSENSE_OFFSET 0 0 0)" />
+  <xacro:property name="rs_rpy"     default="$(optenv DINGO_REALSENSE_RPY 0 0 0)" />
+  <!-- Secondary Realsense Parameters -->
+  <xacro:property name="rs_secondary_enabled" default="$(optenv DINGO_REALSENSE_SECONDARY 0)"/>
+  <xacro:property name="rs_secondary_model"   default="$(optenv DINGO_REALSENSE_SECONDARY_MODEL d435)"/>
+  <xacro:property name="rs_secondary_topic"   default="$(optenv DINGO_REALSENSE_SECONDARY_TOPIC realsense_secondary)" />
+  <xacro:property name="rs_secondary_mount"   default="$(optenv DINGO_REALSENSE_SECONDARY_MOUNT rear)" />
+  <xacro:property name="rs_secondary_prefix"  default="$(optenv DINGO_REALSENSE_SECONDARY_PREFIX ${rs_secondary_mount})" />
+  <xacro:property name="rs_secondary_parent"  default="$(optenv DINGO_REALSENSE_SECONDARY_PARENT ${rs_secondary_mount}_mount)" />
+  <xacro:property name="rs_secondary_xyz"     default="$(optenv DINGO_REALSENSE_SECONDARY_OFFSET 0 0 0)" />
+  <xacro:property name="rs_secondary_rpy"     default="$(optenv DINGO_REALSENSE_SECONDARY_RPY 0 0 ${M_PI})" />
+  <!-- Includes Required for `realsense_sensor` -->
+  <xacro:property name="rs_model"   default="$(optenv DINGO_REALSENSE_MODEL d435)"/>
+  <xacro:if value="${rs_model == 'd435'}">
+    <xacro:include filename="$(find realsense2_description)/urdf/_d435.urdf.xacro" />
+  </xacro:if>
+  <xacro:if value="${rs_model == 'd435i'}">
+    <xacro:include filename="$(find realsense2_description)/urdf/_d435i.urdf.xacro" />
+  </xacro:if>
+  <xacro:if value="${rs_model == 'd415'}">
+    <xacro:include filename="$(find realsense2_description)/urdf/_d415.urdf.xacro" />
+  </xacro:if>
+  <xacro:if value="${rs_model == 'd455'}">
+    <xacro:include filename="$(find realsense2_description)/urdf/_d435.urdf.xacro" />
+  </xacro:if>
+  <xacro:if value="${realsense_enabled}">
+    <xacro:realsense_sensor rs_model="${rs_model}"
+                            prefix="${rs_prefix}"
+                            parent="${rs_parent}"
+                            topic="${rs_topic}">
+      <origin xyz="${rs_xyz}" rpy="${rs_rpy}"/>
+    </xacro:realsense_sensor>
+  </xacro:if>
+  <xacro:if value="${realsense_secondary_enabled}">
+    <xacro:realsense_sensor rs_model="${rs_secondary_model}"
+                            prefix="${rs_secondary_prefix}"
+                            parent="${rs_secondary_parent}"
+                            topic="${rs_secondary_topic}">
+      <origin xyz="${rs_secondary_xyz}" rpy="${rs_secondary_rpy}"/>
+    </xacro:realsense_sensor>
   </xacro:if>
   <!--

File: dingo_description/urdf/accessories/intel_realsense.urdf.xacro (robot description, xacro)
@@ -5,12 +5,35 @@
   gazebo plugin to simulate data from the camera
 -->
+<!-- IMPORTANT NOTE:
+  As of Sept. 2022, due to limitations with the 'realsense2_description' package (see
+  realsense2_description/urdf/_materials.xacro.urdf), the following files must be
+  included in the parent xacro file that will include this one:
+  '''
+  <xacro:if value="${rs_model == 'd435'}">
+    <xacro:include filename="$(find realsense2_description)/urdf/_d435.urdf.xacro" />
+  </xacro:if>
+  <xacro:if value="${rs_model == 'd435i'}">
+    <xacro:include filename="$(find realsense2_description)/urdf/_d435i.urdf.xacro" />
+  </xacro:if>
+  <xacro:if value="${rs_model == 'd415'}">
+    <xacro:include filename="$(find realsense2_description)/urdf/_d415.urdf.xacro" />
+  </xacro:if>
+  <xacro:if value="${rs_model == 'd455'}">
+    <xacro:include filename="$(find realsense2_description)/urdf/_d435.urdf.xacro" />
+  </xacro:if>
+  '''
+  Multiple inclusions of any of these files (even when namespaced), will define
+  the materials at a global level, violating uniqueness property of xacro materials.
+ -->
 <robot xmlns:xacro="http://ros.org/wiki/xacro">
   <xacro:macro name="realsense_sensor" params="
                rs_model:=d435
                prefix:=front
+               parent:=front_mount
                topic:=realsense
                width:=680
                height:=480
-               update_rate:=30">
+               update_rate:=30
+               *origin">
     <xacro:macro name="realsense_gazebo" params="
               prefix=front              model=d4
@@ -80,8 +103,7 @@
     </xacro:macro>
     <xacro:if value="${rs_model == 'd435'}">
-      <xacro:include filename="$(find realsense2_description)/urdf/_d435.urdf.xacro" />
-      <xacro:sensor_d435 parent="${prefix}_mount"
+      <xacro:sensor_d435 parent="${parent}"
                         name="${prefix}_realsense">
-        <origin xyz="$(optenv DINGO_REALSENSE_OFFSET 0 0 0)" rpy="$(optenv DINGO_REALSENSE_RPY 0 0 0)" />
+        <xacro:insert_block name="origin"/>
       </xacro:sensor_d435>
       <xacro:realsense_gazebo
@@ -98,13 +120,12 @@
     </xacro:if>
     <xacro:if value="${rs_model == 'd435i'}">
-      <xacro:include filename="$(find realsense2_description)/urdf/_d435i.urdf.xacro" />
-      <xacro:sensor_d435i parent="$(optenv DINGO_REALSENSE_MOUNT front)_mount"
-                          name="$(optenv DINGO_REALSENSE_MOUNT front)_realsense">
-        <origin xyz="$(optenv DINGO_REALSENSE_OFFSET 0 0 0)" rpy="$(optenv DINGO_REALSENSE_RPY 0 0 0)" />
+      <xacro:sensor_d435i parent="${parent}"
+                          name="${prefix}_realsense">
+        <xacro:insert_block name="origin"/>
       </xacro:sensor_d435i>
       <xacro:realsense_gazebo
-         prefix="$(optenv DINGO_REALSENSE_MOUNT front)"
-         frame="$(optenv DINGO_REALSENSE_MOUNT front)_realsense_link"
-         topic="$(optenv DINGO_REALSENSE_TOPIC realsense)"
+         prefix="${prefix}"
+         frame="${prefix}_realsense_link"
+         topic="${topic}"
          h_fov="1.5184351666666667"
          v_fov="1.0122901111111111"
@@ -123,6 +144,6 @@
           <robotNamespace>/</robotNamespace>
           <updateRate>30.0</updateRate>
-          <bodyName>$(optenv DINGO_REALSENSE_MOUNT front)_realsense_link</bodyName>
-          <topicName>$(optenv DINGO_REALSENSE_TOPIC realsense)/accel/sample</topicName>
+          <bodyName>${prefix}_realsense_link</bodyName>
+          <topicName>${topic}/accel/sample</topicName>
           <accelDrift>0.005 0.005 0.005</accelDrift>
           <accelGaussianNoise>0.005 0.005 0.005</accelGaussianNoise>
@@ -135,6 +156,6 @@
           <robotNamespace>/</robotNamespace>
           <updateRate>30.0</updateRate>
-          <bodyName>$(optenv DINGO_REALSENSE_MOUNT front)_realsense_link</bodyName>
-          <topicName>$(optenv DINGO_REALSENSE_TOPIC realsense)/gyro/sample</topicName>
+          <bodyName>${prefix}_realsense_link</bodyName>
+          <topicName>${topic}/gyro/sample</topicName>
           <accelDrift>0.005 0.005 0.005</accelDrift>
           <accelGaussianNoise>0.005 0.005 0.005</accelGaussianNoise>
@@ -147,13 +168,12 @@
     </xacro:if>
     <xacro:if value="${rs_model == 'd415'}">
-      <xacro:include filename="$(find realsense2_description)/urdf/_d415.urdf.xacro" />
-      <xacro:sensor_d415 parent="$(optenv DINGO_REALSENSE_MOUNT front)_mount"
-                         name="$(optenv DINGO_REALSENSE_MOUNT front)_realsense">
-        <origin xyz="$(optenv DINGO_REALSENSE_OFFSET 0 0 0)" rpy="$(optenv DINGO_REALSENSE_RPY 0 0 0)" />
+      <xacro:sensor_d415 parent="${parent}"
+                         name="${prefix}_realsense">
+        <xacro:insert_block name="origin"/>
       </xacro:sensor_d415>
       <xacro:realsense_gazebo
-         prefix="$(optenv DINGO_REALSENSE_MOUNT front)"
-         frame="$(optenv DINGO_REALSENSE_MOUNT front)_realsense_link"
-         topic="$(optenv DINGO_REALSENSE_TOPIC realsense)"
+         prefix="${prefix}"
+         frame="${prefix}_realsense_link"
+         topic="${topic}"
          h_fov="1.1344640137963142"
          v_fov="0.6981317007977318"
@@ -166,13 +186,12 @@
     <xacro:if value="${rs_model == 'd455'}">
       <!-- TODO: not officially supported yet. Use the D435 mesh for now, even though it's the wrong size -->
-      <xacro:include filename="$(find realsense2_description)/urdf/_d435.urdf.xacro" />
-      <xacro:sensor_d435 parent="$(optenv DINGO_REALSENSE_MOUNT front)_mount"
-                         name="$(optenv DINGO_REALSENSE_MOUNT front)_realsense">
-        <origin xyz="$(optenv DINGO_REALSENSE_OFFSET 0 0 0)" rpy="$(optenv DINGO_REALSENSE_RPY 0 0 0)" />
+      <xacro:sensor_d435 parent="${parent}"
+                         name="${prefix}_realsense">
+        <xacro:insert_block name="origin"/>
       </xacro:sensor_d435>
       <xacro:realsense_gazebo
-         prefix="$(optenv DINGO_REALSENSE_MOUNT front)"
-         frame="$(optenv DINGO_REALSENSE_MOUNT front)_realsense_link"
-         topic="$(optenv DINGO_REALSENSE_TOPIC realsense)"
+         prefix="${prefix}"
+         frame="${prefix}_realsense_link"
+         topic="${topic}"
          h_fov="1.5009831567151233"
          v_fov="0.9948376736367678"
@@ -221,12 +240,12 @@
       </joint>
       <joint type="fixed" name="${prefix}_realsense_mount_joint">
-        <parent link="${prefix}_mount" />
+        <parent link="${parent}" />
         <child link="${prefix}_realsense_bottom_screw_frame" />
         <origin xyz="0 0 0.004" rpy="0 0 0" />
       </joint>
       <xacro:realsense_gazebo
-         prefix="$(optenv DINGO_REALSENSE_MOUNT front)"
-         frame="$(optenv DINGO_REALSENSE_MOUNT front)_realsense_link"
-         topic="$(optenv DINGO_REALSENSE_TOPIC realsense)"
+         prefix="${prefix}"
+         frame="${prefix}_realsense_link"
+         topic="${topic}"
          h_fov="1.2217304763960306"
          v_fov="0.9599310885968813"
