Commit message: Added dingo_control; split dingo_description into separate Dingo-D and Dingo-O flavours; still much work to be done here, but preparing hand-off for Tony

File: dingo_description/dingo_o/urdf/dingo.urdf.xacro (robot description, xacro)
@@ -1,3 +1,7 @@
 <?xml version="1.0"?>
+<!-- TODO(tbaltovski): This is based heavily on the Ridgeback file
+     and may need many updates to reflect the actual dimensions
+     for Dingo-O
+ -->
 <robot name="dingo" xmlns:xacro="http://www.ros.org/wiki/xacro">
   <xacro:macro name="wheel" params="prefix *joint_pose">
@@ -6,5 +10,5 @@
         <origin xyz="0 0 0" rpy="0 0 0"/>
         <geometry>
-          <mesh filename="package://dingo_description/meshes/wheel.dae"/>
+          <mesh filename="package://dingo_description/dingo_o/meshes/wheel.dae"/>
         </geometry>
       </visual>
@@ -12,5 +16,5 @@
         <origin xyz="0 0 0" rpy="0 0 0"/>
         <geometry>
-          <mesh filename="package://dingo_description/meshes/wheel.dae"/>
+          <mesh filename="package://dingo_description/dingo_o/meshes/wheel.dae"/>
         </geometry>
       </collision>
@@ -48,5 +52,5 @@
       <origin xyz="0 0 0" rpy="0 0 0"/>
       <geometry>
-        <mesh filename="package://dingo_description/meshes/body.dae"/>
+        <mesh filename="package://dingo_description/dingo_o/meshes/body.dae"/>
       </geometry>
     </visual>
@@ -54,5 +58,5 @@
       <origin xyz="0 0 0"/>
       <geometry>
-        <mesh filename="package://dingo_description/meshes/body_collision.stl"/>
+        <mesh filename="package://dingo_description/dingo_o/meshes/body_collision.stl"/>
       </geometry>
     </collision>
