Commit message: Updated dingo_description for dingo-d simulation

File: dingo_description/urdf/accessories/hokuyo_ust10.urdf.xacro (robot description, xacro)
@@ -53,5 +53,5 @@
         <geometry>
           <!-- Origin of this mesh is the base of the bracket. -->
-          <mesh filename="package://dingo_description/meshes/hokuyo_ust10.stl" />
+          <mesh filename="file://$(find dingo_description)/meshes/hokuyo_ust10.stl" />
         </geometry>
         <material name="dark_grey" />

File: dingo_description/urdf/accessories/sick_lms1xx_mount.urdf.xacro (robot description, xacro)
@@ -34,5 +34,5 @@
         <geometry>
           <!-- Origin of this mesh is the base of the bracket. -->
-          <mesh filename="package://dingo_description/meshes/sick-lms1xx-bracket.stl" />
+          <mesh filename="file://$(find dingo_description)/meshes/sick-lms1xx-bracket.stl" />
         </geometry>
         <material name="dark_grey" />

File: dingo_description/urdf/dingo-d.urdf.xacro (robot description, xacro)
@@ -18,5 +18,5 @@
         <origin xyz="0 0 0" rpy="0 0 0"/>
         <geometry>
-          <mesh filename="package://dingo_description/meshes/wheel.stl"/>
+          <mesh filename="file://$(find dingo_description)/meshes/wheel.stl"/>
         </geometry>
         <material name="black" />
@@ -52,13 +52,4 @@
       <axis xyz="0 1 0" />
     </joint>
-    <transmission name="${prefix}_wheel_trans">
-      <type>transmission_interface/SimpleTransmission</type>
-      <joint name="${prefix}_wheel">
-        <hardwareInterface>hardware_interface/VelocityJointInterface</hardwareInterface>
-      </joint>
-      <actuator name="${prefix}_actuator">
-        <mechanicalReduction>1</mechanicalReduction>
-      </actuator>
-    </transmission>
   </xacro:macro>
   <xacro:wheel prefix="left">
@@ -125,5 +116,5 @@
       <origin xyz="0 0 0" rpy="0 0 0"/>
       <geometry>
-        <mesh filename="package://dingo_description/meshes/diff_chassis.dae"/>
+        <mesh filename="file://$(find dingo_description)/meshes/diff_chassis.dae"/>
       </geometry>
     </visual>
@@ -131,5 +122,5 @@
       <origin xyz="0 0 0"/>
       <geometry>
-        <mesh filename="package://dingo_description/meshes/diff_chassis_collision.stl"/>
+        <mesh filename="file://$(find dingo_description)/meshes/diff_chassis_collision.stl"/>
       </geometry>
     </collision>
@@ -138,5 +129,5 @@
       <origin xyz="0 0 0" rpy="0 0 0"/>
       <mass value="10.0"/>
-      <!-- Moments of inertia: ( chassis without wheels ) -->
+      <!-- Moments of inertia ( chassis without wheels ) -->
       <inertia
         ixx="0.2216" ixy="0" ixz="0"
@@ -215,10 +206,32 @@
     <child link="front_bumper_mount" />
   </joint>
+	<!-- ROS 2 control -->
+	<ros2_control name="dingo-d_hardware" type="system">
+		<hardware>
+			<plugin>gazebo_ros2_control/GazeboSystem</plugin>
+		</hardware>
+		<joint name="left_wheel">
+			<command_interface name="velocity">
+				<param name="min">-10</param>
+				<param name="max">10</param>
+			</command_interface>
+			<state_interface name="position"/>
+			<state_interface name="velocity"/>
+		</joint>
+		<joint name="right_wheel">
+			<command_interface name="velocity">
+				<param name="min">-10</param>
+				<param name="max">10</param>
+			</command_interface>
+			<state_interface name="position"/>
+			<state_interface name="velocity"/>
+		</joint>
+	</ros2_control>
   <!-- Bring in simulation data for Gazebo. -->
   <xacro:include filename="$(find dingo_description)/urdf/dingo.gazebo" />
+	<xacro:include filename="$(find dingo_description)/urdf/dingo-d.gazebo" />
   <!-- Optional standard accessories, including their simulation data. The rendering
        of these into the final description is controlled by optenv variables, which
        default each one to off.-->
-  <xacro:include filename="$(find dingo_description)/urdf/accessories.urdf.xacro" />
   <!-- Optional custom includes. -->
   <xacro:include filename="$(optenv DINGO_URDF_EXTRAS empty.urdf)" />

File: dingo_description/urdf/dingo-o.urdf.xacro (robot description, xacro)
@@ -75,5 +75,5 @@
       <origin xyz="0 0 0" rpy="0 0 0"/>
       <geometry>
-        <mesh filename="package://dingo_description/meshes/omni_chassis.dae"/>
+        <mesh filename="file://$(find dingo_description)/meshes/omni_chassis.dae"/>
       </geometry>
       <material name="dark_grey" />
@@ -82,5 +82,5 @@
       <origin xyz="0 0 0"/>
       <geometry>
-        <mesh filename="package://dingo_description/meshes/omni_chassis_collision.stl"/>
+        <mesh filename="file://$(find dingo_description)/meshes/omni_chassis_collision.stl"/>
       </geometry>
     </collision>
